File: Hardware/Prototyp/Automatischer-Kabelschneider/main_microcontroller_AKS.kicad_sch (KiCad schematic)
At the start: 1 part, among them U2 ESP32-S3-WROOM-2

Commit message: 20240410
Parts:
- added C1: 100n, Capacitor_SMD:C_0805_2012Metric, symbol Device:C
- added C4: 1u, Capacitor_SMD:C_0805_2012Metric, symbol Device:C
Changed lines of the file:
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@@
+		)
+	)
+	(symbol
+		(lib_id "Device:C")
+		(at 113.03 74.93 0)
+		(unit 1)
+		(exclude_from_sim no)
+		(in_bom yes)
+		(on_board yes)
+		(dnp no)
+		(fields_autoplaced yes)
+		(property "Reference" "C1"
+			(at 116.84 73.6599 0)
+			(effects
+				(font
+					(size 1.27 1.27)
+				)
+				(justify left)
+			)
+		)
+		(property "Value" "100n"
+			(at 116.84 76.1999 0)
+			(effects
+				(font
+					(size 1.27 1.27)
+				)
+				(justify left)
+			)
+		)
+		(property "Footprint" "Capacitor_SMD:C_0805_2012Metric"
+			(at 113.9952 78.74 0)
+			(effects
+				(font
+					(size 1.27 1.27)
+				)
+				(hide yes)
+			)
+		)
+		(property "Datasheet" "~"
+			(at 113.03 74.93 0)
+			(effects
+				(font
+					(size 1.27 1.27)
+				)
+				(hide yes)
+			)
+		)
+		(property "Description" "Unpolarized capacitor"
+			(at 113.03 74.93 0)
+			(effects
+				(font
+					(size 1.27 1.27)
+				)
+				(hide yes)
+			)
+		)
+		(pin "1"
+		)
+		(pin "2"
+		)
+		(instances
+			(project "Automatischer-Kabelschneider"
+				(path "/ff414881-00bc-48a3-bd83-dba8c1da722a/352ad1d3-9b58-40da-b881-d99a3f860b8b"
+					(reference "C1")
+					(unit 1)
+				)
+			)
+		)
+	)
+	(symbol
+		(lib_id "Device:C")
+		(at 106.68 74.93 0)
+		(mirror y)
+		(unit 1)
+		(exclude_from_sim no)
+		(in_bom yes)
+		(on_board yes)
+		(dnp no)
+		(property "Reference" "C4"
+			(at 102.87 73.6599 0)
+			(effects
+				(font
+					(size 1.27 1.27)
+				)
+				(justify left)
+			)
+		)
+		(property "Value" "1u"
+			(at 102.87 76.1999 0)
+			(effects
+				(font
+					(size 1.27 1.27)
+				)
+				(justify left)
+			)
+		)
+		(property "Footprint" "Capacitor_SMD:C_0805_2012Metric"
+			(at 105.7148 78.74 0)
+			(effects
+				(font
+					(size 1.27 1.27)
+				)
+				(hide yes)
+			)
+		)
+		(property "Datasheet" "~"
+			(at 106.68 74.93 0)
+			(effects
+				(font
+					(size 1.27 1.27)
+				)
+				(hide yes)
+			)
+		)
+		(property "Description" "Unpolarized capacitor"
+			(at 106.68 74.93 0)
+			(effects
+				(font
+					(size 1.27 1.27)
+				)
+				(hide yes)
+			)
+		)
+		(pin "1"
+		)
+		(pin "2"
+		)
+		(instances
+			(project "Automatischer-Kabelschneider"
+				(path "/ff414881-00bc-48a3-bd83-dba8c1da722a/352ad1d3-9b58-40da-b881-d99a3f860b8b"
+					(reference "C4")
+					(unit 1)
+				)
+			)
 		)
 	)

Commit message: 20240415
Parts:
- added C15: 1u, Capacitor_SMD:C_0805_2012Metric, symbol Device:C
- added D6, D7, D8, D9: WS2812B-2020, LED_SMD:LED_WS2812B-2020_PLCC4_2.0x2.0mm, symbol LED:WS2812B-2020
- added J3: Conn_01x05, Connector_PinHeader_2.54mm:PinHeader_1x05_P2.54mm_Vertical, symbol Connector_Generic:Conn_01x05
- added R7: 10k, Resistor_SMD:R_0805_2012Metric, symbol Device:R
- added SW1, SW2: SW_Push, Button_Switch_SMD:SW_Push_1P1T_NO_6x6mm_H9.5mm, symbol Switch:SW_Push
- added TP7: TestPoint_Small, TestPoint:TestPoint_Pad_D1.0mm, symbol Connector:TestPoint_Small
- C13: renamed from C4; value 1u -> 22u
- renumbered C1 to C14, U2 to U4
Connections:
- net GND: now reaches U4.1 (GND), U4.40 (GND), U4.41 (GND)
- net GND: now also C13.2, C14.2, C15.2, SW1.2, SW2.1
- net D-: now reaches U4.13 (USB_D-/IO19)
- net D+: now reaches U4.14 (USB_D+/IO20)
- net +3.3V: now reaches U4.2 (3V3)
- net +3.3V: now also C13.1, C14.1, R7.1
- net at U4.27 (IO0): now also SW1.1
- net at U4.3 (EN): now also C15.1, R7.2, SW2.2
- new net: D9.1 (DOUT), TP7.1
- new net: D8.1 (DOUT), D9.3 (DIN)
- new net: D7.1 (DOUT), D8.3 (DIN)
- new net: D6.1 (DOUT), D7.3 (DIN)
Other:
- moved on the sheet: C13, C14, U4

Commit message: 20240418
Parts:
- removed D6, D7, D8, D9: WS2812B-2020, LED_SMD:LED_WS2812B-2020_PLCC4_2.0x2.0mm, symbol LED:WS2812B-2020
- removed J3: Conn_01x05, Connector_PinHeader_2.54mm:PinHeader_1x05_P2.54mm_Vertical, symbol Connector_Generic:Conn_01x05
- removed TP7: TestPoint_Small, TestPoint:TestPoint_Pad_D1.0mm, symbol Connector:TestPoint_Small
- added J5: Conn_02x05_Odd_Even, Connector_PinHeader_1.27mm:PinHeader_2x05_P1.27mm_Vertical, symbol Connector_Generic:Conn_02x05_Odd_Even
- added JP1: SolderJumper_3_Bridged12, Jumper:SolderJumper-3_P1.3mm_Bridged12_RoundedPad1.0x1.5mm, symbol Jumper:SolderJumper_3_Bridged12
- added R8: 10k, Resistor_SMD:R_0805_2012Metric, symbol Device:R
- added TP8, TP9: TestPoint_Small, TestPoint:TestPoint_Pad_D1.0mm, symbol Connector:TestPoint_Small
- added U5, U6: TMC2209_SILENTSTEPSTICK, TMC2209_Module:MODULE_TMC2209_SILENTSTEPSTICK, symbol TMC2209_SILENTSTEPSTICK:TMC2209_SILENTSTEPSTICK
Connections:
- net +3.3V: now also JP1.1 (A)
- net GND: now also JP1.3 (B)
- net PROG_SEL: now reaches U4.15 (IO3)
- net PROG_SEL: now also R8.2
- net at U4.16 (IO46): now also TP8.1
- net at U4.26 (IO45): now also TP9.1
- net BOOT: now reaches SW1.1, U4.27 (IO0)
- new net: U6.1 (GND), U6.7 (GND)
- new net: JP1.2 (C), R8.1
- new net: U5.1 (GND), U5.7 (GND)
Other:
- moved on the sheet: SW1

Commit message: 20240501
Parts:
- added D10, D11, D12, D13: WS2812B-2020, LED_SMD:LED_WS2812B-2020_PLCC4_2.0x2.0mm, symbol LED:WS2812B-2020
- added TP10, TP11, TP12: TestPoint_Small, TestPoint:TestPoint_Pad_D1.0mm, symbol Connector:TestPoint_Small
Connections:
- net +3.3V: now also J5.1 (Pin_1), D10.4 (VDD), D11.4 (VDD), D12.4 (VDD), D13.4 (VDD)
- net GND: now also J5.3 (Pin_3), J5.5 (Pin_5), J5.7 (Pin_7), J5.9 (Pin_9), D10.2 (VSS), D11.2 (VSS), D12.2 (VSS), D13.2 (VSS)
- net MTMS: now reaches J5.2 (Pin_2)
- net MTMS: now also U4.35 (MTMS/IO42)
- net MTCK: now reaches J5.4 (Pin_4)
- net MTCK: now also U4.32 (MTCK/IO39)
- net MTDO: now reaches J5.6 (Pin_6)
- net MTDO: now also U4.33 (MTDO/IO40)
- net MTDI: now reaches J5.8 (Pin_8)
- net MTDI: now also U4.34 (MTDI/IO41)
- net at U4.36 (RXD0/IO44): now also TP11.1
- net at U4.37 (TXD0/IO43): now also TP10.1
- new net: D12.1 (DOUT), D13.3 (DIN)
- new net: D11.1 (DOUT), D12.3 (DIN)
- new net: D13.1 (DOUT), TP12.1
- new net: D10.1 (DOUT), D11.3 (DIN)
- no-connect marks 0 -> 1
Other:
- moved on the sheet: J5

Commit message: Schematic completed
Parts:
- added C19, C20, C21, C22: 22u, Capacitor_SMD:C_0805_2012Metric, symbol Device:C
- added J3, J5: Conn_01x04, Connector_Phoenix_GMSTB:PhoenixContact_GMSTBA_2,5_4-G-7,62_1x04_P7.62mm_Horizontal, symbol Connector_Generic:Conn_01x04
- added Q3, Q4: Q_NMOS_GSD, Package_TO_SOT_SMD:TSOT-23, symbol Device:Q_NMOS_GSD
- added R10, R11, R9: 10k, Resistor_SMD:R_0805_2012Metric, symbol Device:R
- added TP11, TP12: TestPoint_Small, TestPoint:TestPoint_Pad_D1.0mm, symbol Connector:TestPoint_Small
- renumbered C13 to C16, C14 to C17, C15 to C18, D10 to D6, D11 to D7, D12 to D8, D13 to D9, J5 to J4, SW2 to SW1, SW1 to SW2, TP8 to TP10, TP12 to TP13, TP10 to TP7, TP11 to TP8, U4 to U6, U6 to U7
Connections:
- net +3.3V: now also R8.2, U5.14 (MS2), U5.15 (MS1), U5.2 (VIO), U7.14 (MS2), U7.15 (MS1), U7.2 (VIO), C19.1, C21.1, Q3.1 (G), Q4.1 (G), R10.2
- net GND: now also U5.1 (GND), U5.11 (PDN), U5.13 (SPRD), U5.7 (GND), U7.1 (GND), U7.11 (PDN), U7.13 (SPRD), U7.7 (GND), C19.2, C20.2, C21.2, C22.2
- net MD2_STEP: now reaches U7.10 (STEP)
- net MD2_STEP: now also U6.6 (IO6)
- net MD2_!EN: now reaches U7.16 (~{EN})
- net MD2_!EN: now also U6.38 (IO2)
- net at U7.3 (M1B): now also J5.2 (Pin_2)
- net at U7.4 (M1A): now also J5.4 (Pin_4)
- net at U7.5 (M2A): now also J5.3 (Pin_3)
- net at U7.6 (M2B): now also J5.1 (Pin_1)
- net +20V: now reaches U7.8 (VM)
- net +20V: now also U5.8 (VM), C20.1, C22.1
- net MD2_DIR: now reaches U7.9 (DIR)
- net MD2_DIR: now also U6.7 (IO7)
- net WS2812: now reaches U6.12 (IO8)
- net WS2812: now also D6.3 (DIN)
- net ESP_Tx: now reaches U6.23 (IO21)
- net ESP_Tx: now also R8.1, Q3.2 (S)
- net at U6.24 (IO47): now also TP11.1
- net at U6.25 (IO48): now also TP12.1
- net ESP_Rx: now reaches U6.31 (IO38)
- net ESP_Rx: now also Q4.2 (S), R10.1
- net MD1_!EN: now reaches U6.39 (IO1)
- net MD1_!EN: now also U5.16 (~{EN})
- net MD1_STEP: now reaches U6.4 (IO4)
- net MD1_STEP: now also U5.10 (STEP)
- net MD1_DIR: now reaches U6.5 (IO5)
- net MD1_DIR: now also U5.9 (DIR)
- net at JP1.2 (C): now also U6.15 (IO3); no longer R8.1
- net at U5.3 (M1B): now also J3.2 (Pin_2)
- net at U5.4 (M1A): now also J3.4 (Pin_4)
- net at U5.5 (M2A): now also J3.3 (Pin_3)
- net at U5.6 (M2B): now also J3.1 (Pin_1)
- removed net PROG_SEL: R8.2, U6.15 (IO3)
- new net +5V: R11.2, R9.2
- new net 5V_ESP_Rx: Q4.3 (D), R11.1
- new net 5V_ESP_Tx: Q3.3 (D), R9.1
- no-connect marks 1 -> 17
Other:
- note added: "https://learn.watterott.com/de/silentstepstick/"
- moved on the sheet: C16, C17, C18, D6, D7, D8, D9, J4, JP1, R7, SW1, SW2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

Commit message: PCB finished
Parts:
- added J4: Conn_01x02, Connector_Wire:SolderWire-1.5sqmm_1x02_P6mm_D1.7mm_OD3mm_Relief, symbol Connector_Generic:Conn_01x02
- added J5: Conn_02x05_Odd_Even, Connector_IDC:IDC-Header_2x05_P2.54mm_Vertical, symbol Connector_Generic:Conn_02x05_Odd_Even
- renumbered J5 to J6, J4 to J7, U5 to U6, U6 to U7, U7 to U8
Connections:
- net +3.3V: now also J5.9 (Pin_9)
- net GND: now also J5.10 (Pin_10)
- net IO17: now reaches U7.10 (IO17)
- net IO17: now also J5.7 (Pin_7)
- net IO18: now reaches U7.11 (IO18)
- net IO18: now also J5.8 (Pin_8)
- net Touch1: now reaches U7.17 (IO9)
- net Touch1: now also J4.1 (Pin_1)
- net Touch2: now reaches U7.18 (IO10)
- net Touch2: now also J4.2 (Pin_2)
- net IO11: now reaches U7.19 (IO11)
- net IO11: now also J5.1 (Pin_1)
- net IO12: now reaches U7.20 (IO12)
- net IO12: now also J5.2 (Pin_2)
- net IO13: now reaches U7.21 (IO13)
- net IO13: now also J5.3 (Pin_3)
- net IO14: now reaches U7.22 (IO14)
- net IO14: now also J5.4 (Pin_4)
- net EN: now reaches C18.1, R7.2, SW1.2, U7.3 (EN)
- net IO15: now reaches U7.8 (IO15)
- net IO15: now also J5.5 (Pin_5)
- net IO16: now reaches U7.9 (IO16)
- net IO16: now also J5.6 (Pin_6)
- no-connect marks 17 -> 7
Other:
- moved on the sheet: C16, C17, C18, C19, C20, C21, C22, J3, J6, J7, JP1, Q3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
