File: Hardware/Prototyp/Automatischer-Kabelschneider/Automatischer-Kabelschneider.kicad_pcb (KiCad board)
At the start: 4 copper layers, 4 parts, among them J1 USB_C_Receptacle_USB2.0_16P, U1 AP63203WU, U2 ESP32-S3-WROOM-2

Commit message: 20240410
Parts:
- removed L1: 3u9, Inductor_SMD:L_Wuerth_MAPI-4020
- added C1: 100n, Capacitor_SMD:C_0805_2012Metric, F.Cu at (63.9, 71.7)
- added C2: 470u, Capacitor_SMD:C_Elec_8x10.2, F.Cu at (36.3, 50.0)
- added C3: 470u, Capacitor_SMD:C_Elec_8x10.2, F.Cu at (36.3, 59.8)
- added C4: 1u, Capacitor_SMD:C_0805_2012Metric, F.Cu at (63.9, 74.7)
- added D2: D_TVS, Diode_SMD:D_0603_1608Metric, F.Cu at (31.5, 70.5)
- added D3: D_TVS, Diode_SMD:D_0603_1608Metric, F.Cu at (31.5, 73.1)
- added D4: D_TVS, Diode_SMD:D_0603_1608Metric, F.Cu at (31.5, 75.6)
- added D5: D_TVS, Diode_SMD:D_0603_1608Metric, F.Cu at (31.5, 78.2)
- added J2: USB_C_Receptacle_USB2.0_16P, Connector_USB:USB_C_Receptacle_GCT_USB4105-xx-A_16P_TopMnt_Horizontal, F.Cu at (48.7, 75.4)
- added U5: TVS2200DRV, Package_SON:WSON-6-1EP_2x2mm_P0.65mm_EP1x1.6mm, F.Cu at (35.6, 71.0)
- J1: value USB_C_Receptacle_USB2.0_16P -> Conn_01x04; footprint Connector_USB:USB_C_Receptacle_GCT_USB4105-xx-A_16P_TopMnt_Horizontal -> Connector_Phoenix_GMSTB:PhoenixContact_GMSTBA_2,5_4-G-7,62_1x04_P7.62mm_Horizontal
- U1: value AP63203WU -> CYPD3177-24LQ; footprint Package_TO_SOT_SMD:TSOT-23-6 -> Package_DFN_QFN:QFN-24-1EP_4x4mm_P0.5mm_EP2.75x2.75mm
- moved J1 47.5 mm to (34.5, 34.0)
- moved U1 20.2 mm to (46.0, 83.3)

Commit message: 20240411
Parts:
- removed C3: 470u, Capacitor_SMD:C_Elec_8x10.2
- added C10: 1u, Capacitor_SMD:C_0805_2012Metric, F.Cu at (93.3, 97.0)
- added C11: 1u, Capacitor_SMD:C_0805_2012Metric, F.Cu at (93.3, 100.0)
- added C5: 1u, Capacitor_SMD:C_0805_2012Metric, F.Cu at (93.3, 81.9)
- added C6: 100n, Capacitor_SMD:C_0805_2012Metric, F.Cu at (93.3, 84.9)
- added C7: 3u3, Capacitor_SMD:C_0805_2012Metric, F.Cu at (93.3, 87.9)
- added C8: 1u, Capacitor_SMD:C_0805_2012Metric, F.Cu at (93.3, 90.9)
- added C9: 100n, Capacitor_SMD:C_0805_2012Metric, F.Cu at (93.3, 94.0)
- added D1: gr, Diode_SMD:D_0805_2012Metric, F.Cu at (93.3, 103.0)
- added Q1: IRF540N, Package_TO_SOT_THT:TO-220-3_Horizontal_TabDown, F.Cu at (71.2, 100.6)
- added Q2: IRF540N, Package_TO_SOT_THT:TO-220-3_Horizontal_TabDown, F.Cu at (82.7, 100.6)
- added R1: 1k, Resistor_SMD:R_0805_2012Metric, F.Cu at (97.7, 81.9)
- added R3: 10k, Resistor_SMD:R_0805_2012Metric, F.Cu at (97.7, 84.8)
- added R4: 50k, Resistor_SMD:R_0805_2012Metric, F.Cu at (97.7, 87.8)
- added R5: 5k1, Resistor_SMD:R_0805_2012Metric, F.Cu at (97.7, 90.7)
- added R6: 5k1, Resistor_SMD:R_0805_2012Metric, F.Cu at (97.7, 93.7)
- added R7: 1k, Resistor_SMD:R_0805_2012Metric, F.Cu at (97.7, 96.6)
- U5: value TVS2200DRV -> TVS220x
Connections:
- J1 pad 1: +20V -> VBUS
- J1 pad 2: GND -> +20V
- U1 pad 1: unconnected-(U1-VBUS_MIN-Pad1) -> VDDD
- U1 pad 18: unconnected-(U1-VBUS_IN-Pad18) -> VBUS
- U1 pad 19: Net-(U1-GND-Pad19) -> GND
- U1 pad 2: unconnected-(U1-VBUS_MAX-Pad2) -> VDDD
- U1 pad 22: Net-(U1-GND-Pad19) -> GND
- U1 pad 23: unconnected-(U1-VDDD-Pad23) -> VDDD
- U1 pad 24: unconnected-(U1-VCCD-Pad24) -> VCCD
- U1 pad 25: Net-(U1-GND-Pad19) -> GND
- U1 pad 3: unconnected-(U1-VBUS_FET_EN-Pad3) -> Net-(U1-VBUS_FET_EN)
- U1 pad 5: unconnected-(U1-ISNK_COARSE-Pad5) -> Net-(U1-ISNK_COARSE)
- U1 pad 6: unconnected-(U1-ISNK_FINE-Pad6) -> GND
- U1 pad 9: unconnected-(U1-FAULT-Pad9) -> Net-(D1-K)

Commit message: 20240415
Parts:
- added C10: 10u, Capacitor_SMD:C_0805_2012Metric, F.Cu at (32.5, 108.2)
- added C11: 22u, Capacitor_SMD:C_0805_2012Metric, F.Cu at (32.5, 111.2)
- added C12: 22u, Capacitor_SMD:C_0805_2012Metric, F.Cu at (32.5, 114.2)
- added C15: 100n, Capacitor_SMD:C_0805_2012Metric, F.Cu at (127.2, 87.1)
- added C9: 100n, Capacitor_SMD:C_0805_2012Metric, F.Cu at (32.5, 105.1)
- added H1: MountingHole, MountingHole:MountingHole_3.2mm_M3, F.Cu at (26.3, 107.6)
- added H2: MountingHole, MountingHole:MountingHole_3.2mm_M3, F.Cu at (26.3, 115.6)
- added H3: MountingHole, MountingHole:MountingHole_3.2mm_M3, F.Cu at (26.3, 123.5)
- added H4: MountingHole, MountingHole:MountingHole_3.2mm_M3, F.Cu at (26.3, 131.5)
- added L1: 3u9, Inductor_SMD_Wurth:L_Wurth_WE-LQSH-4020, F.Cu at (33.2, 124.6)
- added R7: 10k, Resistor_SMD:R_0805_2012Metric, F.Cu at (127.2, 90.1)
- added SW1: SW_Push, Button_Switch_SMD:SW_Push_1P1T_NO_6x6mm_H9.5mm, F.Cu at (119.5, 89.4)
- added SW2: SW_Push, Button_Switch_SMD:SW_Push_1P1T_NO_6x6mm_H9.5mm, F.Cu at (119.5, 96.9)
- added TP1: TestPoint_Small, TestPoint:TestPoint_Pad_D1.0mm, F.Cu at (31.8, 117.2)
- added TP2: TestPoint_Small, TestPoint:TestPoint_Pad_D1.0mm, F.Cu at (31.8, 120.3)
- added TP3: TestPoint_Small, TestPoint:TestPoint_Pad_D1.0mm, F.Cu at (34.9, 117.2)
- added TP4: TestPoint_Small, TestPoint:TestPoint_Pad_D1.0mm, F.Cu at (34.9, 120.3)
- added TP5: TestPoint_Small, TestPoint:TestPoint_Pad_D1.0mm, F.Cu at (37.9, 117.2)
- added TP6: TestPoint_Small, TestPoint:TestPoint_Pad_D1.0mm, F.Cu at (37.9, 120.3)
- added U3: AP63203WU, Package_TO_SOT_SMD:TSOT-23-6, F.Cu at (32.9, 129.7)
- C13: renamed from C4; value 1u -> 22u
- renumbered C10 to C1, C1 to C14, C11 to C2, C5 to C3, C7 to C4, C8 to C5, C9 to C7, C2 to C8, J2 to J1, J1 to J2, R5 to R1, R3 to R2, R4 to R3, R6 to R4, R7 to R5, R1 to R6, U5 to U1, U1 to U2, U2 to U4
Connections:
- net Net-(Q1-G) renamed /Powersupply_AKS/GATE
- C13 pad 1: unconnected-(C4-Pad1) -> +3.3V
- C13 pad 2: unconnected-(C4-Pad2) -> GND
- C14 pad 1: unconnected-(C1-Pad1) -> +3.3V
- C14 pad 2: unconnected-(C1-Pad2) -> GND
- D4 pad 2: /Powersupply_AKS/D- -> /Main Microcontroller/D-
- D5 pad 2: /Powersupply_AKS/D+ -> /Main Microcontroller/D+
- J1 pad A6: /Powersupply_AKS/D+ -> /Main Microcontroller/D+
- J1 pad A7: /Powersupply_AKS/D- -> /Main Microcontroller/D-
- J1 pad B6: /Powersupply_AKS/D+ -> /Main Microcontroller/D+
- J1 pad B7: /Powersupply_AKS/D- -> /Main Microcontroller/D-
- U2 pad 10: unconnected-(U1-FLIP-Pad10) -> Net-(U2-FLIP)
- U2 pad 11: unconnected-(U1-VDC_OUT-Pad11) -> +20V
- U2 pad 12: unconnected-(U1-HPI_SDA-Pad12) -> Net-(U2-HPI_SDA)
- U2 pad 13: unconnected-(U1-HPI_SCL-Pad13) -> Net-(U2-HPI_SCL)
- U2 pad 4: unconnected-(U1-SAFE_PWR_EN-Pad4) -> Net-(U2-SAFE_PWR_EN)
- U2 pad 7: unconnected-(U1-~{HPI_INT}-Pad7) -> Net-(U2-~{HPI_INT})
- U2 pad 8: unconnected-(U1-GPIO_1-Pad8) -> Net-(U2-GPIO_1)
- U4 pad 1: Net-(U2-GND-Pad1) -> GND
- U4 pad 13: unconnected-(U2-USB_D-/IO19-Pad13) -> /Main Microcontroller/D-
- U4 pad 14: unconnected-(U2-USB_D+/IO20-Pad14) -> /Main Microcontroller/D+
- U4 pad 2: unconnected-(U2-3V3-Pad2) -> +3.3V
- U4 pad 27: unconnected-(U2-IO0-Pad27) -> Net-(U4-IO0)
- U4 pad 3: unconnected-(U2-EN-Pad3) -> Net-(U4-EN)
- U4 pad 40: Net-(U2-GND-Pad1) -> GND
- U4 pad 41: Net-(U2-GND-Pad1) -> GND

Commit message: 20240418
Parts:
- added C16: 100n, Capacitor_SMD:C_0805_2012Metric, F.Cu at (50.6, 120.2)
- added C17: 10u, Capacitor_SMD:C_0805_2012Metric, F.Cu at (50.6, 123.2)
- added C18: 22u, Capacitor_SMD:C_0805_2012Metric, F.Cu at (50.6, 126.3)
- added C19: 22u, Capacitor_SMD:C_0805_2012Metric, F.Cu at (50.6, 129.3)
- added C20: 22u, Capacitor_SMD:C_0805_2012Metric, F.Cu at (62.9, 120.2)
- added C21: 100n, Capacitor_SMD:C_0805_2012Metric, F.Cu at (62.9, 123.2)
- added D6: WS2812B-2020, LED_SMD:LED_WS2812B-2020_PLCC4_2.0x2.0mm, F.Cu at (168.6, 84.1)
- added D7: WS2812B-2020, LED_SMD:LED_WS2812B-2020_PLCC4_2.0x2.0mm, F.Cu at (168.6, 87.7)
- added D8: WS2812B-2020, LED_SMD:LED_WS2812B-2020_PLCC4_2.0x2.0mm, F.Cu at (168.6, 91.2)
- added D9: WS2812B-2020, LED_SMD:LED_WS2812B-2020_PLCC4_2.0x2.0mm, F.Cu at (168.6, 94.8)
- added J3: Conn_01x05, Connector_PinHeader_2.54mm:PinHeader_1x05_P2.54mm_Vertical, F.Cu at (168.8, 103.1)
- added J4: Conn_02x05_Odd_Even, Connector_PinHeader_1.27mm:PinHeader_2x05_P1.27mm_Vertical, F.Cu at (150.4, 109.5)
- added J5: Conn_02x05_Odd_Even, Connector_PinHeader_1.27mm:PinHeader_2x05_P1.27mm_Vertical, F.Cu at (142.9, 109.5)
- added JP1: SolderJumper_3_Bridged12, Jumper:SolderJumper-3_P1.3mm_Bridged12_RoundedPad1.0x1.5mm, F.Cu at (144.5, 93.8)
- added L2: 4u7, Inductor_SMD_Wurth:L_Wurth_WE-LQSH-4020, F.Cu at (55.7, 121.5)
- added R8: 10k, Resistor_SMD:R_0805_2012Metric, F.Cu at (138.8, 95.8)
- added TP7: TestPoint_Small, TestPoint:TestPoint_Pad_D1.0mm, F.Cu at (168.1, 98.1)
- added TP8: TestPoint_Small, TestPoint:TestPoint_Pad_D1.0mm, F.Cu at (143.2, 87.5)
- added TP9: TestPoint_Small, TestPoint:TestPoint_Pad_D1.0mm, F.Cu at (143.2, 90.5)
- added U5: TMC2209_SILENTSTEPSTICK, TMC2209_Module:MODULE_TMC2209_SILENTSTEPSTICK, F.Cu at (157.0, 69.4)
- added U6: TMC2209_SILENTSTEPSTICK, TMC2209_Module:MODULE_TMC2209_SILENTSTEPSTICK, F.Cu at (174.3, 69.4)
- added U7: AP63205WU, Package_TO_SOT_SMD:TSOT-23-6, F.Cu at (56.5, 128.7)
- added U8: ATmega2560-16A, Package_QFP:TQFP-100_14x14mm_P0.5mm, F.Cu at (124.0, 123.8)
- C15: value 100n -> 1u
Connections:
- net Net-(U4-IO0) renamed /Main Microcontroller/BOOT
- J2 pad 1: VBUS -> +20V
- J2 pad 2: +20V -> +5V
- U4 pad 15: unconnected-(U4-IO3-Pad15) -> /Main Microcontroller/PROG_SEL
- U4 pad 16: unconnected-(U4-IO46-Pad16) -> Net-(U4-IO46)
- U4 pad 26: unconnected-(U4-IO45-Pad26) -> Net-(U4-IO45)

Commit message: 20240501
Parts:
- added C22: 100n, Capacitor_SMD:C_0805_2012Metric, F.Cu at (91.0, 120.3)
- added C23: 100n, Capacitor_SMD:C_0805_2012Metric, F.Cu at (91.0, 123.3)
- added C24: 100n, Capacitor_SMD:C_0805_2012Metric, F.Cu at (91.0, 126.3)
- added C25: 100n, Capacitor_SMD:C_0805_2012Metric, F.Cu at (91.0, 129.3)
- added C26: 100n, Capacitor_SMD:C_0805_2012Metric, F.Cu at (91.0, 132.4)
- added C27: 100n, Capacitor_SMD:C_0805_2012Metric, F.Cu at (91.0, 135.4)
- added L3: 10u, Inductor_SMD:L_0805_2012Metric, F.Cu at (99.9, 127.8)
- added R10: 10k, Resistor_SMD:R_0805_2012Metric, F.Cu at (95.4, 130.8)
- added R9: 0r, Resistor_SMD:R_0805_2012Metric, F.Cu at (95.4, 127.9)
- added SW3: SW_Push, Button_Switch_SMD:SW_Push_1P1T_NO_6x6mm_H9.5mm, F.Cu at (98.7, 122.6)
Connections:
- net Net-(U2-ISNK_COARSE) renamed /Powersupply_AKS/ISNK_COARSE
- net Net-(U2-VBUS_FET_EN) renamed /Powersupply_AKS/VBUS_FET_EN
- C20 pad 1: unconnected-(C20-Pad1) -> +5V
- C20 pad 2: unconnected-(C20-Pad2) -> GND
- C21 pad 1: unconnected-(C21-Pad1) -> +5V
- C21 pad 2: unconnected-(C21-Pad2) -> GND
- U8 pad 10: Net-(U8-VCC-Pad10) -> +5V
- U8 pad 100: unconnected-(U8-AVCC-Pad100) -> VDDA
- U8 pad 11: Net-(U8-GND-Pad11) -> GND
- U8 pad 30: unconnected-(U8-~{RESET}-Pad30) -> Net-(U8-~{RESET})
- U8 pad 31: Net-(U8-VCC-Pad10) -> +5V
- U8 pad 32: Net-(U8-GND-Pad11) -> GND
- U8 pad 61: Net-(U8-VCC-Pad10) -> +5V
- U8 pad 62: Net-(U8-GND-Pad11) -> GND
- U8 pad 80: Net-(U8-VCC-Pad10) -> +5V
- U8 pad 81: Net-(U8-GND-Pad11) -> GND
- U8 pad 98: unconnected-(U8-AREF-Pad98) -> Net-(U8-AREF)
- U8 pad 99: Net-(U8-GND-Pad11) -> GND

Commit message: Schematic completed
Parts:
- removed the C8 at (36.3, 50.0)
- added C19: 22u, Capacitor_SMD:C_0805_2012Metric, F.Cu at (186.5, 70.1)
- added C20: 22u, Capacitor_SMD:C_0805_2012Metric, F.Cu at (192.1, 64.6)
- added C21: 22u, Capacitor_SMD:C_0805_2012Metric, F.Cu at (186.5, 67.1)
- added C22: 22u, Capacitor_SMD:C_0805_2012Metric, F.Cu at (192.1, 73.7)
- added C25: 18p, Capacitor_SMD:C_0805_2012Metric, F.Cu at (327.0, 104.5)
- added C26: 18p, Capacitor_SMD:C_0805_2012Metric, F.Cu at (327.0, 107.5)
- added D6: WS2812B-2020, LED_SMD:LED_WS2812B-2020_PLCC4_2.0x2.0mm, F.Cu at (102.1, 162.0)
- added D7: WS2812B-2020, LED_SMD:LED_WS2812B-2020_PLCC4_2.0x2.0mm, F.Cu at (102.1, 165.6)
- added D8: WS2812B-2020, LED_SMD:LED_WS2812B-2020_PLCC4_2.0x2.0mm, F.Cu at (102.1, 169.1)
- added D9: WS2812B-2020, LED_SMD:LED_WS2812B-2020_PLCC4_2.0x2.0mm, F.Cu at (102.1, 172.7)
- added J3: Conn_01x04, Connector_Phoenix_GMSTB:PhoenixContact_GMSTBA_2,5_4-G-7,62_1x04_P7.62mm_Horizontal, F.Cu at (77.0, 111.3)
- added J5: Conn_01x04, Connector_Phoenix_GMSTB:PhoenixContact_GMSTBA_2,5_4-G-7,62_1x04_P7.62mm_Horizontal, F.Cu at (77.0, 125.8)
- added J6: Conn_02x05_Odd_Even, Connector_IDC:IDC-Header_2x05_P2.54mm_Vertical, F.Cu at (388.6, 76.7)
- added J7: Conn_02x05_Odd_Even, Connector_IDC:IDC-Header_2x05_P2.54mm_Vertical, F.Cu at (408.9, 153.9)
- added J8: Conn_02x05_Odd_Even, Connector_IDC:IDC-Header_2x05_P2.54mm_Vertical, F.Cu at (373.3, 154.3)
- added Q3: Q_NMOS_GSD, Package_TO_SOT_SMD:TSOT-23, F.Cu at (320.0, 132.1)
- added Q4: Q_NMOS_GSD, Package_TO_SOT_SMD:TSOT-23, F.Cu at (320.0, 127.4)
- added Q5: Q_NMOS_GSD, Package_TO_SOT_SMD:TSOT-23, F.Cu at (327.4, 127.4)
- added Q6: Q_NMOS_GSD, Package_TO_SOT_SMD:TSOT-23, F.Cu at (327.4, 132.1)
- added R10: 10k, Resistor_SMD:R_0805_2012Metric, F.Cu at (94.4, 87.5)
- added R11: 10k, Resistor_SMD:R_0805_2012Metric, F.Cu at (94.4, 90.4)
- added R14: 10k, Resistor_SMD:R_0805_2012Metric, F.Cu at (315.7, 139.5)
- added R15: 10k, Resistor_SMD:R_0805_2012Metric, F.Cu at (315.7, 142.4)
- added R16: 1k, Resistor_SMD:R_0805_2012Metric, F.Cu at (315.7, 154.2)
- added R17: 2k, Resistor_SMD:R_0805_2012Metric, F.Cu at (315.7, 151.3)
- added R18: 10k, Resistor_SMD:R_0805_2012Metric, F.Cu at (315.7, 145.4)
- added R19: 10k, Resistor_SMD:R_0805_2012Metric, F.Cu at (315.7, 148.3)
- added R9: 10k, Resistor_SMD:R_0805_2012Metric, F.Cu at (94.4, 84.5)
- added TP11: TestPoint_Small, TestPoint:TestPoint_Pad_D1.0mm, F.Cu at (195.8, 64.7)
- added TP12: TestPoint_Small, TestPoint:TestPoint_Pad_D1.0mm, F.Cu at (195.8, 67.7)
- added TP13: TestPoint_Small, TestPoint:TestPoint_Pad_D1.0mm, F.Cu at (105.7, 167.9)
- added TP14: TestPoint_Small, TestPoint:TestPoint_Pad_D1.0mm, F.Cu at (394.5, 116.8)
- added TP15: TestPoint_Small, TestPoint:TestPoint_Pad_D1.0mm, F.Cu at (392.9, 115.3)
- added TP16: TestPoint_Small, TestPoint:TestPoint_Pad_D1.0mm, F.Cu at (394.5, 113.8)
- added TP17: TestPoint_Small, TestPoint:TestPoint_Pad_D1.0mm, F.Cu at (392.9, 112.3)
- added TP18: TestPoint_Small, TestPoint:TestPoint_Pad_D1.0mm, F.Cu at (394.5, 110.7)
- added TP19: TestPoint_Small, TestPoint:TestPoint_Pad_D1.0mm, F.Cu at (392.9, 109.2)
- added TP20: TestPoint_Small, TestPoint:TestPoint_Pad_D1.0mm, F.Cu at (394.5, 107.7)
- added TP21: TestPoint_Small, TestPoint:TestPoint_Pad_D1.0mm, F.Cu at (392.9, 106.2)
- added TP22: TestPoint_Small, TestPoint:TestPoint_Pad_D1.0mm, F.Cu at (361.7, 100.1)
- added TP23: TestPoint_Small, TestPoint:TestPoint_Pad_D1.0mm, F.Cu at (363.2, 101.6)
- added TP24: TestPoint_Small, TestPoint:TestPoint_Pad_D1.0mm, F.Cu at (361.7, 103.1)
- added TP25: TestPoint_Small, TestPoint:TestPoint_Pad_D1.0mm, F.Cu at (363.2, 104.6)
- added TP26: TestPoint_Small, TestPoint:TestPoint_Pad_D1.0mm, F.Cu at (361.7, 106.2)
- added TP27: TestPoint_Small, TestPoint:TestPoint_Pad_D1.0mm, F.Cu at (363.2, 107.7)
- added TP28: TestPoint_Small, TestPoint:TestPoint_Pad_D1.0mm, F.Cu at (361.7, 109.2)
- added TP29: TestPoint_Small, TestPoint:TestPoint_Pad_D1.0mm, F.Cu at (363.2, 110.7)
- added TP30: TestPoint_Small, TestPoint:TestPoint_Pad_D1.0mm, F.Cu at (370.3, 85.9)
- added TP32: TestPoint_Small, TestPoint:TestPoint_Pad_D1.0mm, F.Cu at (370.3, 88.9)
- added TP33: TestPoint_Small, TestPoint:TestPoint_Pad_D1.0mm, F.Cu at (363.2, 130.6)
- added TP34: TestPoint_Small, TestPoint:TestPoint_Pad_D1.0mm, F.Cu at (370.3, 92.0)
- added TP35: TestPoint_Small, TestPoint:TestPoint_Pad_D1.0mm, F.Cu at (363.2, 121.4)
- added TP36: TestPoint_Small, TestPoint:TestPoint_Pad_D1.0mm, F.Cu at (370.3, 95.0)
- added TP37: TestPoint_Small, TestPoint:TestPoint_Pad_D1.0mm, F.Cu at (363.2, 124.5)
- added TP38: TestPoint_Small, TestPoint:TestPoint_Pad_D1.0mm, F.Cu at (363.2, 127.5)
- added TP7: TestPoint_Small, TestPoint:TestPoint_Pad_D1.0mm, F.Cu at (105.7, 161.8)
- added TP8: TestPoint_Small, TestPoint:TestPoint_Pad_D1.0mm, F.Cu at (105.7, 164.8)
- added Y1: 16M, Crystal:Crystal_SMD_ECS_CSM3X-2Pin_7.6x4.1mm, F.Cu at (330.0, 100.2)
- moved U8 253.1 mm to (376.8, 109.7)
- moved C28 253.0 mm to (315.1, 101.1)
- moved C29 253.0 mm to (315.1, 104.1)
- moved L3 250.8 mm to (349.6, 104.1)
- moved C23 250.8 mm to (340.7, 105.6)
- moved C24 250.8 mm to (340.7, 108.7)
- moved C27 250.8 mm to (340.7, 111.7)
- moved C30 250.8 mm to (340.7, 96.6)
- moved C31 250.8 mm to (340.7, 99.6)
- moved C32 250.8 mm to (340.7, 102.6)
- moved R12 250.8 mm to (345.1, 107.1)
- moved R13 250.8 mm to (345.1, 104.2)
- moved SW3 250.8 mm to (348.4, 98.9)
- moved D10 246.8 mm to (414.0, 110.7)
- moved D11 246.8 mm to (414.0, 114.3)
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- renumbered C11 to C10, C12 to C11, C16 to C12, C17 to C13, C18 to C14, C19 to C15, C13 to C16, C14 to C17, C15 to C18, C25 to C23, C26 to C24, C20 to C28, C21 to C29, C22 to C30, C23 to C31, C24 to C32, C9 to C8, C10 to C9, D6 to D10, D7 to D11, D8 to D12, D9 to D13, J3 to J10, J5 to J4, J4 to J9, R10 to R12, R9 to R13, SW2 to SW1, SW1 to SW2, TP8 to TP10, TP7 to TP31, U7 to U4, U4 to U6, U6 to U7
Connections:
- D10 pad 2: unconnected-(D6-VSS-Pad2) -> GND
- D10 pad 3: unconnected-(D6-DIN-Pad3) -> PD5
- D10 pad 4: unconnected-(D6-VDD-Pad4) -> +5V
- D11 pad 2: unconnected-(D7-VSS-Pad2) -> GND
- D11 pad 4: unconnected-(D7-VDD-Pad4) -> +5V
- D12 pad 2: unconnected-(D8-VSS-Pad2) -> GND
- D12 pad 4: unconnected-(D8-VDD-Pad4) -> +5V
- D13 pad 2: unconnected-(D9-VSS-Pad2) -> GND
- D13 pad 4: unconnected-(D9-VDD-Pad4) -> +5V
- J10 pad 1: unconnected-(J3-Pin_1-Pad1) -> Net-(J10-Pin_1)
- J10 pad 2: unconnected-(J3-Pin_2-Pad2) -> DISP_SDA
- J10 pad 3: unconnected-(J3-Pin_3-Pad3) -> DISP_SCL
- J10 pad 4: unconnected-(J3-Pin_4-Pad4) -> +3.3V
- J10 pad 5: unconnected-(J3-Pin_5-Pad5) -> GND
- J4 pad 1: unconnected-(J5-Pin_1-Pad1) -> +3.3V
- J4 pad 2: unconnected-(J5-Pin_2-Pad2) -> MTMS
- J4 pad 3: unconnected-(J5-Pin_3-Pad3) -> GND
- J4 pad 4: unconnected-(J5-Pin_4-Pad4) -> MTCK
- J4 pad 5: unconnected-(J5-Pin_5-Pad5) -> GND
- J4 pad 6: unconnected-(J5-Pin_6-Pad6) -> MTDO
- J4 pad 7: unconnected-(J5-Pin_7-Pad7) -> GND
- J4 pad 8: unconnected-(J5-Pin_8-Pad8) -> MTDI
- J4 pad 9: unconnected-(J5-Pin_9-Pad9) -> GND
- J9 pad 1: unconnected-(J4-Pin_1-Pad1) -> ATMEGA_TCK
- J9 pad 10: unconnected-(J4-Pin_10-Pad10) (its old number) -> GND
- J9 pad 2: unconnected-(J4-Pin_2-Pad2) -> GND
- J9 pad 3: unconnected-(J4-Pin_3-Pad3) -> ATMEGA_TDO
- J9 pad 4: unconnected-(J4-Pin_4-Pad4) -> +5V
- J9 pad 5: unconnected-(J4-Pin_5-Pad5) -> ATMEGA_TMS
- J9 pad 6: unconnected-(J4-Pin_6-Pad6) -> ATMEGA_RST
- J9 pad 7: unconnected-(J4-Pin_7-Pad7) -> ATMEGA_!WR
- J9 pad 8: unconnected-(J4-Pin_8-Pad8) -> ATMEGA_!RD
- J9 pad 9: unconnected-(J4-Pin_9-Pad9) -> ATMEGA_TDI
- R12 pad 2: Net-(U8-~{RESET}) -> ATMEGA_RST
- R8 pad 1: Net-(JP1-C) -> /Main Microcontroller/ESP_Tx
- R8 pad 2: /Main Microcontroller/PROG_SEL -> +3.3V
- SW3 pad 2: Net-(U8-~{RESET}) -> ATMEGA_RST
- U5 pad 1: Net-(U5-GND-Pad1) -> GND
- U5 pad 10: unconnected-(U5-STEP-Pad10) -> MD1_STEP
- U5 pad 11: unconnected-(U5-PDN-Pad11) -> GND
- U5 pad 13: unconnected-(U5-SPRD-Pad13) -> GND
- U5 pad 14: unconnected-(U5-MS2-Pad14) -> +3.3V
- U5 pad 15: unconnected-(U5-MS1-Pad15) -> +3.3V
- U5 pad 16: unconnected-(U5-~{EN}-Pad16) -> MD1_!EN
- U5 pad 2: unconnected-(U5-VIO-Pad2) -> +3.3V
- U5 pad 3: unconnected-(U5-M1B-Pad3) -> Net-(J3-Pin_2)
- U5 pad 4: unconnected-(U5-M1A-Pad4) -> Net-(J3-Pin_4)
- U5 pad 5: unconnected-(U5-M2A-Pad5) -> Net-(J3-Pin_3)
- U5 pad 6: unconnected-(U5-M2B-Pad6) -> Net-(J3-Pin_1)
- U5 pad 7: Net-(U5-GND-Pad1) -> GND
- U5 pad 8: unconnected-(U5-VM-Pad8) -> +20V
- U5 pad 9: unconnected-(U5-DIR-Pad9) -> MD1_DIR
- U6 pad 12: unconnected-(U4-IO8-Pad12) -> WS2812
- U6 pad 15: /Main Microcontroller/PROG_SEL -> Net-(JP1-C)
- U6 pad 23: unconnected-(U4-IO21-Pad23) -> /Main Microcontroller/ESP_Tx
- U6 pad 24: unconnected-(U4-IO47-Pad24) -> Net-(U6-IO47)
- U6 pad 25: unconnected-(U4-IO48-Pad25) -> Net-(U6-IO48)
- U6 pad 31: unconnected-(U4-IO38-Pad31) -> /Main Microcontroller/ESP_Rx
- U6 pad 32: unconnected-(U4-MTCK/IO39-Pad32) -> MTCK
- U6 pad 33: unconnected-(U4-MTDO/IO40-Pad33) -> MTDO
- U6 pad 34: unconnected-(U4-MTDI/IO41-Pad34) -> MTDI
- U6 pad 35: unconnected-(U4-MTMS/IO42-Pad35) -> MTMS
- U6 pad 36: unconnected-(U4-RXD0/IO44-Pad36) -> Net-(U6-RXD0/IO44)
- U6 pad 37: unconnected-(U4-TXD0/IO43-Pad37) -> Net-(U6-TXD0/IO43)
- U6 pad 38: unconnected-(U4-IO2-Pad38) -> MD2_!EN
- U6 pad 39: unconnected-(U4-IO1-Pad39) -> MD1_!EN
- U6 pad 4: unconnected-(U4-IO4-Pad4) -> MD1_STEP
- U6 pad 5: unconnected-(U4-IO5-Pad5) -> MD1_DIR
- U6 pad 6: unconnected-(U4-IO6-Pad6) -> MD2_STEP
- U6 pad 7: unconnected-(U4-IO7-Pad7) -> MD2_DIR
- U7 pad 1: Net-(U6-GND-Pad1) -> GND
- U7 pad 10: unconnected-(U6-STEP-Pad10) -> MD2_STEP
- U7 pad 11: unconnected-(U6-PDN-Pad11) -> GND
- U7 pad 13: unconnected-(U6-SPRD-Pad13) -> GND
- U7 pad 14: unconnected-(U6-MS2-Pad14) -> +3.3V
- U7 pad 15: unconnected-(U6-MS1-Pad15) -> +3.3V
- U7 pad 16: unconnected-(U6-~{EN}-Pad16) -> MD2_!EN
- U7 pad 2: unconnected-(U6-VIO-Pad2) -> +3.3V
- U7 pad 3: unconnected-(U6-M1B-Pad3) -> Net-(J5-Pin_2)
- U7 pad 4: unconnected-(U6-M1A-Pad4) -> Net-(J5-Pin_4)
- U7 pad 5: unconnected-(U6-M2A-Pad5) -> Net-(J5-Pin_3)
- U7 pad 6: unconnected-(U6-M2B-Pad6) -> Net-(J5-Pin_1)
- U7 pad 7: Net-(U6-GND-Pad1) -> GND
- U7 pad 8: unconnected-(U6-VM-Pad8) -> +20V
- U7 pad 9: unconnected-(U6-DIR-Pad9) -> MD2_DIR
- U8 pad 1: unconnected-(U8-PG5-Pad1) -> Net-(U8-PG5)
- U8 pad 19: unconnected-(U8-PB0-Pad19) -> /Slave Microcontroller/PB0
- U8 pad 2: unconnected-(U8-PE0-Pad2) -> Net-(U8-PE0)
- U8 pad 20: unconnected-(U8-PB1-Pad20) -> /Slave Microcontroller/PB1
- U8 pad 21: unconnected-(U8-PB2-Pad21) -> /Slave Microcontroller/PB2
- U8 pad 22: unconnected-(U8-PB3-Pad22) -> /Slave Microcontroller/PB3
- U8 pad 23: unconnected-(U8-PB4-Pad23) -> /Slave Microcontroller/PB4
- U8 pad 24: unconnected-(U8-PB5-Pad24) -> /Slave Microcontroller/PB5
- U8 pad 25: unconnected-(U8-PB6-Pad25) -> /Slave Microcontroller/PB6
- U8 pad 26: unconnected-(U8-PB7-Pad26) -> /Slave Microcontroller/PB7
- U8 pad 28: unconnected-(U8-PG3-Pad28) -> Net-(U8-PG3)
- U8 pad 29: unconnected-(U8-PG4-Pad29) -> Net-(U8-PG4)
- U8 pad 3: unconnected-(U8-PE1-Pad3) -> Net-(U8-PE1)
- U8 pad 30: Net-(U8-~{RESET}) -> ATMEGA_RST
- U8 pad 33: unconnected-(U8-XTAL2-Pad33) -> Net-(U8-XTAL2)
- U8 pad 34: unconnected-(U8-XTAL1-Pad34) -> Net-(U8-XTAL1)
- U8 pad 4: unconnected-(U8-PE2-Pad4) -> Net-(U8-PE2)
- U8 pad 43: unconnected-(U8-PD0-Pad43) -> ATMEGA_SCL
- U8 pad 44: unconnected-(U8-PD1-Pad44) -> ATMEGA_SDA
- U8 pad 45: unconnected-(U8-PD2-Pad45) -> /Slave Microcontroller/ATMEGA_Rx
- U8 pad 46: unconnected-(U8-PD3-Pad46) -> /Slave Microcontroller/ATMEGA_Tx
- U8 pad 47: unconnected-(U8-PD4-Pad47) -> AT_DISP_RST
- U8 pad 48: unconnected-(U8-PD5-Pad48) -> PD5
- U8 pad 49: unconnected-(U8-PD6-Pad49) -> /Slave Microcontroller/PD6
- U8 pad 5: unconnected-(U8-PE3-Pad5) -> Net-(U8-PE3)
- U8 pad 50: unconnected-(U8-PD7-Pad50) -> /Slave Microcontroller/PD7
- U8 pad 51: unconnected-(U8-PG0-Pad51) -> ATMEGA_!WR
- U8 pad 52: unconnected-(U8-PG1-Pad52) -> ATMEGA_!RD
- U8 pad 53: unconnected-(U8-PC0-Pad53) -> Net-(U8-PC0)
- U8 pad 54: unconnected-(U8-PC1-Pad54) -> Net-(U8-PC1)
- U8 pad 55: unconnected-(U8-PC2-Pad55) -> Net-(U8-PC2)
- U8 pad 56: unconnected-(U8-PC3-Pad56) -> Net-(U8-PC3)
- U8 pad 57: unconnected-(U8-PC4-Pad57) -> Net-(U8-PC4)
- U8 pad 58: unconnected-(U8-PC5-Pad58) -> Net-(U8-PC5)
- U8 pad 59: unconnected-(U8-PC6-Pad59) -> Net-(U8-PC6)
- U8 pad 6: unconnected-(U8-PE4-Pad6) -> Net-(U8-PE4)
- U8 pad 60: unconnected-(U8-PC7-Pad60) -> Net-(U8-PC7)
- U8 pad 7: unconnected-(U8-PE5-Pad7) -> Net-(U8-PE5)
- U8 pad 70: unconnected-(U8-PG2-Pad70) -> Net-(U8-PG2)
- U8 pad 71: unconnected-(U8-PA7-Pad71) -> /Slave Microcontroller/PA7
- U8 pad 72: unconnected-(U8-PA6-Pad72) -> /Slave Microcontroller/PA6
- U8 pad 73: unconnected-(U8-PA5-Pad73) -> /Slave Microcontroller/PA5
- U8 pad 74: unconnected-(U8-PA4-Pad74) -> /Slave Microcontroller/PA4
- U8 pad 75: unconnected-(U8-PA3-Pad75) -> /Slave Microcontroller/PA3
- U8 pad 76: unconnected-(U8-PA2-Pad76) -> /Slave Microcontroller/PA2
- U8 pad 77: unconnected-(U8-PA1-Pad77) -> /Slave Microcontroller/PA1
- U8 pad 78: unconnected-(U8-PA0-Pad78) -> /Slave Microcontroller/PA0
- U8 pad 8: unconnected-(U8-PE6-Pad8) -> Net-(U8-PE6)
- U8 pad 9: unconnected-(U8-PE7-Pad9) -> Net-(U8-PE7)
- U8 pad 90: unconnected-(U8-PF7-Pad90) -> ATMEGA_TDI
- U8 pad 91: unconnected-(U8-PF6-Pad91) -> ATMEGA_TDO
- U8 pad 92: unconnected-(U8-PF5-Pad92) -> ATMEGA_TMS
- U8 pad 93: unconnected-(U8-PF4-Pad93) -> ATMEGA_TCK
- U8 pad 94: unconnected-(U8-PF3-Pad94) -> Net-(U8-PF3)
- U8 pad 95: unconnected-(U8-PF2-Pad95) -> Net-(U8-PF2)
- U8 pad 96: unconnected-(U8-PF1-Pad96) -> Net-(U8-PF1)
- U8 pad 97: unconnected-(U8-PF0-Pad97) -> Net-(U8-PF0)
Routing:
- net Net-(U8-PC7): track 0.00 -> 0.84 mm

Commit message: PCB finished
Parts:
- added J4: Conn_01x02, Connector_Wire:SolderWire-1.5sqmm_1x02_P6mm_D1.7mm_OD3mm_Relief, F.Cu at (98.8, 69.3)
- added J5: Conn_02x05_Odd_Even, Connector_IDC:IDC-Header_2x05_P2.54mm_Vertical, F.Cu at (70.8, 43.7)
- added U1: TVS220x, Package_SON:WSON-6-1EP_2x2mm_P0.65mm_EP1x1.6mm, F.Cu at (73.6, 129.3)
- Q1, Q2: footprint Package_TO_SOT_THT:TO-220-3_Horizontal_TabDown -> Package_TO_SOT_THT:TO-220-3_Vertical
- TP10, TP11, TP12, TP7, TP8, TP9: moved to B.Cu
- moved J9 280.3 mm to (129.2, 136.1), turned to 90 degrees
- moved TP31 255.1 mm to (171.9, 42.9), turned to 90 degrees
- moved D13 251.9 mm to (174.4, 43.4)
- moved D12 247.5 mm to (178.0, 43.4)
- moved D11 243.0 mm to (181.5, 43.4)
- moved D10 238.6 mm to (185.1, 43.4)
- moved R13 234.9 mm to (110.9, 122.7)
- moved TP38 231.3 mm to (137.5, 76.9)
- moved TP22 226.7 mm to (136.0, 78.5)
- moved TP23 226.7 mm to (137.5, 80.0)
- moved TP24 226.7 mm to (136.0, 81.5)
- moved TP25 226.7 mm to (137.5, 83.0)
- moved TP26 226.7 mm to (136.0, 84.6)
- moved TP27 226.7 mm to (137.5, 86.1)
- moved TP28 226.7 mm to (136.0, 87.6)
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- renumbered J8 to J10, J9 to J11, J10 to J12, J5 to J6, J4 to J7, J6 to J8, J7 to J9, U1 to U2, U2 to U3, U3 to U4, U4 to U5, U5 to U6, U6 to U7, U7 to U8, U8 to U9
Connections:
- net Net-(U6-EN) renamed /Main Microcontroller/EN
- C27 pad 1: Net-(U8-AREF) -> VDDA
- J8 pad 5: /Slave Microcontroller/PA3 -> /Slave Microcontroller/PA4
- U7 pad 10: unconnected-(U6-IO17-Pad10) -> /Main Microcontroller/IO17
- U7 pad 11: unconnected-(U6-IO18-Pad11) -> /Main Microcontroller/IO18
- U7 pad 17: unconnected-(U6-IO9-Pad17) -> /Main Microcontroller/Touch1
- U7 pad 18: unconnected-(U6-IO10-Pad18) -> /Main Microcontroller/Touch2
- U7 pad 19: unconnected-(U6-IO11-Pad19) -> /Main Microcontroller/IO11
- U7 pad 20: unconnected-(U6-IO12-Pad20) -> /Main Microcontroller/IO12
- U7 pad 21: unconnected-(U6-IO13-Pad21) -> /Main Microcontroller/IO13
- U7 pad 22: unconnected-(U6-IO14-Pad22) -> /Main Microcontroller/IO14
- U7 pad 8: unconnected-(U6-IO15-Pad8) -> /Main Microcontroller/IO15
- U7 pad 9: unconnected-(U6-IO16-Pad9) -> /Main Microcontroller/IO16
- U9 pad 98: Net-(U8-AREF) -> VDDA
Routing:
- net +5V: track 0.00 -> 479.3 mm, vias 0 -> 14
- net +3.3V: track 0.00 -> 456.1 mm, vias 0 -> 10
- net /Main Microcontroller/D+: track 0.00 -> 148.4 mm, vias 0 -> 2
- net /Main Microcontroller/D-: track 0.00 -> 147.2 mm, vias 0 -> 2
- net GND: track 0.00 -> 145.3 mm, vias 0 -> 37
- net +20V: track 0.00 -> 134.9 mm, vias 0 -> 1
- net /Slave Microcontroller/ATMEGA_Tx: track 0.00 -> 117.1 mm, vias 0 -> 5
- net /Slave Microcontroller/ATMEGA_Rx: track 0.00 -> 116.6 mm, vias 0 -> 5
- net PD5: track 0.00 -> 103.0 mm, vias 0 -> 2
- net GNDREF: track 0.00 -> 101.0 mm, vias 0 -> 6
- net MD2_!EN: track 0.00 -> 90.5 mm, vias 0 -> 2
- net ATMEGA_RST: track 0.00 -> 81.2 mm, vias 0 -> 2
- net AT_DISP_RST: track 0.00 -> 70.8 mm, vias 0 -> 2
- net MD1_!EN: track 0.00 -> 70.4 mm, vias 0 -> 2
- net /Main Microcontroller/IO14: track 0.00 -> 68.9 mm, vias 0 -> 3
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- added copper zone on F.Cu, net +20V
- added copper zone on F.Cu, net +3.3V
- added copper zone on F.Cu, net +5V
- added copper zone on B.Cu, net GND
- added copper zone on F.Cu, net GND
- added copper zone on In1.Cu, net GND
- added copper zone on In2.Cu, net GND
- added copper zone on F.Cu, net Net-(U4-SW)
- added copper zone on F.Cu, net Net-(U5-SW)
- added copper zone on F.Cu, net VBUS
Other:
- board outline added: 160 x 100 mm
