File: Hardware/Prototyp/Automatischer-Kabelschneider/Automatischer-Kabelschneider.kicad_pcb (KiCad board)
At the start: 4 copper layers, 160 x 100 mm, 141 parts, among them J1 USB_C_Receptacle_USB2.0_16P, J10 Conn_02x05_Odd_Even, J11 Conn_02x05_Odd_Even, J12 Conn_01x05, J2 Conn_01x04, J3 Conn_01x04, J4 Conn_01x02, J5 Conn_02x05_Odd_Even, J6 Conn_01x04, J7 Conn_02x05_Odd_Even, J8 Conn_02x05_Odd_Even, J9 Conn_02x05_Odd_Even, Q1 IRF540N, Q2 IRF540N, Q3 Q_NMOS_GSD, Q4 Q_NMOS_GSD, Q5 Q_NMOS_GSD, Q6 Q_NMOS_GSD, SW1 SW_Push, SW2 SW_Push, SW3 SW_Push, U1 TVS220x, U2 TVS220x, U3 CYPD3177-24LQ, U4 AP63203WU, U5 AP63205WU, U6 TMC2209_SILENTSTEPSTICK, U7 ESP32-S3-WROOM-2, U8 TMC2209_SILENTSTEPSTICK, U9 ATmega2560-16A, Y1 16M

Commit message: Prototype PCB finished
Parts:
- Y1: footprint Crystal:Crystal_SMD_ECS_CSM3X-2Pin_7.6x4.1mm -> Crystal:Crystal_SMD_HC49-SD
- moved SW3 1.45 mm to (179.8, 127.2)
- moved C26 0.38 mm to (187.5, 128.5)
- moved C25 0.37 mm to (192.1, 128.5)
Connections:
- C27 pad 1: VDDA -> Net-(U9-AREF)
- U9 pad 98: VDDA -> Net-(U9-AREF)
Routing:
- net VDDA: track 14.5 -> 7.56 mm
- net Net-(U9-AREF): track 0.00 -> 3.62 mm
- net ATMEGA_SDA: track 53.3 -> 55.3 mm
- net Net-(U9-XTAL2): track 16.7 -> 18.0 mm
- net Net-(U9-XTAL1): track 16.9 -> 18.1 mm
- net ATMEGA_RST: track 81.2 -> 82.3 mm
- net +20V: track 163.0 -> 163.9 mm
- net GNDREF: track 101.0 -> 101.9 mm
- net GND: vias 37 -> 164
Other:
- board text added: "3V3 REGULATOR"
- board text added: "5V REGULATOR"
- board text added: "M1A M2A M1B M2B"
- board text added: "Prototyp Automatischer Kabelschneider Huruvarshan und Adrian Rev. 1.0"
- board text added: "RESET SDA SCL 3V3 GND"
- board text added: "Touch1"
- board text added: "Touch2"
