File: Hardware/Prototyp/Automatischer-Kabelschneider/slave_microcontroller_AKS.kicad_sch (KiCad schematic)
At the start: 0 parts

Commit message: 20240418
Parts:
- added C20: 22u, Capacitor_SMD:C_0805_2012Metric, symbol Device:C
- added C21, C22, C23, C24, C25, C26, C27: 100n, Capacitor_SMD:C_0805_2012Metric, symbol Device:C
- added D6, D7, D8, D9: WS2812B-2020, LED_SMD:LED_WS2812B-2020_PLCC4_2.0x2.0mm, symbol LED:WS2812B-2020
- added J3: Conn_01x05, Connector_PinHeader_2.54mm:PinHeader_1x05_P2.54mm_Vertical, symbol Connector_Generic:Conn_01x05
- added J4: Conn_02x05_Odd_Even, Connector_PinHeader_1.27mm:PinHeader_2x05_P1.27mm_Vertical, symbol Connector_Generic:Conn_02x05_Odd_Even
- added L3: 10u, Inductor_SMD:L_0805_2012Metric, symbol Device:L
- added R10: 10k, Resistor_SMD:R_0805_2012Metric, symbol Device:R
- added R9: 0r, Resistor_SMD:R_0805_2012Metric, symbol Device:R
- added SW3: SW_Push, Button_Switch_SMD:SW_Push_1P1T_NO_6x6mm_H9.5mm, symbol Switch:SW_Push
- added TP7: TestPoint_Small, TestPoint:TestPoint_Pad_D1.0mm, symbol Connector:TestPoint_Small
- added U8: ATmega2560-16A, Package_QFP:TQFP-100_14x14mm_P0.5mm, symbol MCU_Microchip_ATmega:ATmega2560-16A
Connections:
- new net: D9.1 (DOUT), TP7.1
- new net: D8.1 (DOUT), D9.3 (DIN)
- new net: D7.1 (DOUT), D8.3 (DIN)
- new net: D6.1 (DOUT), D7.3 (DIN)
- new net: C27.1, U8.98 (AREF)
- new net: R10.2, SW3.2, U8.30 (~{RESET})
- new net +5V: C20.1, C21.1, C22.1, C23.1, C24.1, C25.1, L3.1, R10.1, U8.10 (VCC), U8.31 (VCC), U8.61 (VCC), U8.80 (VCC)
- new net GND: C20.2, C21.2, C22.2, C23.2, C24.2, C25.2, R9.1, SW3.1, U8.11 (GND), U8.32 (GND), U8.62 (GND), U8.81 (GND), U8.99 (GND)
- new net GNDREF: C26.2, C27.2, R9.2
- new net VDDA: C26.1, L3.2, U8.100 (AVCC)
Other:
- note added: "i2c disp"
- note added: "jtag"

Commit message: 20240501
Parts:
- added C28, C29: 18p, Capacitor_SMD:C_0805_2012Metric, symbol Device:C
- added Y1: 16M, Crystal:Crystal_SMD_ECS_CSM3X-2Pin_7.6x4.1mm, symbol Device:Crystal
Connections:
- net +3.3V: now also J3.4 (Pin_4)
- net +5V: now also D6.4 (VDD), D7.4 (VDD), D8.4 (VDD), D9.4 (VDD), J4.4 (Pin_4)
- net GND: now also D6.2 (VSS), D7.2 (VSS), D8.2 (VSS), D9.2 (VSS), J3.5 (Pin_5), J4.10 (Pin_10), J4.2 (Pin_2)
- net GNDREF: now also C28.1, C29.1
- net ATMEGA_RST: now reaches R10.2, SW3.2, U8.30 (~{RESET})
- net ATMEGA_RST: now also J4.6 (Pin_6)
- net at U8.33 (XTAL2): now also C29.2, Y1.1
- net at U8.34 (XTAL1): now also C28.2, Y1.2
- net ATMEGA_!WR: now reaches U8.51 (PG0)
- net ATMEGA_!WR: now also J4.7 (Pin_7)
- net ATMEGA_!RD: now reaches U8.52 (PG1)
- net ATMEGA_!RD: now also J4.8 (Pin_8)
- net ATMEGA_TDI: now reaches U8.90 (PF7)
- net ATMEGA_TDI: now also J4.9 (Pin_9)
- net ATMEGA_TDO: now reaches U8.91 (PF6)
- net ATMEGA_TDO: now also J4.3 (Pin_3)
- net ATMEGA_TMS: now reaches U8.92 (PF5)
- net ATMEGA_TMS: now also J4.5 (Pin_5)
- net ATMEGA_TCK: now reaches U8.93 (PF4)
- net ATMEGA_TCK: now also J4.1 (Pin_1)
Other:
- note removed: "i2c disp"
- note removed: "jtag"
- moved on the sheet: C25, C26, C27, D6, D7, D8, D9, J3, J4, L3, R9, TP7

Commit message: Schematic completed
Parts:
- added J6, J7, J8: Conn_02x05_Odd_Even, Connector_IDC:IDC-Header_2x05_P2.54mm_Vertical, symbol Connector_Generic:Conn_02x05_Odd_Even
- added Q5, Q6: Q_NMOS_GSD, Package_TO_SOT_SMD:TSOT-23, symbol Device:Q_NMOS_GSD
- added R14, R15, R18, R19: 10k, Resistor_SMD:R_0805_2012Metric, symbol Device:R
- added R16: 1k, Resistor_SMD:R_0805_2012Metric, symbol Device:R
- added R17: 2k, Resistor_SMD:R_0805_2012Metric, symbol Device:R
- added TP14, TP15, TP16, TP17, TP18, TP19, TP20, TP21, TP22, TP23, TP24, TP25, TP26, TP27, TP28, TP29, TP30, TP32, TP33, TP34, TP35, TP36, TP37, TP38: TestPoint_Small, TestPoint:TestPoint_Pad_D1.0mm, symbol Connector:TestPoint_Small
- renumbered C25 to C23, C26 to C24, C28 to C25, C29 to C26, C20 to C28, C21 to C29, C22 to C30, C23 to C31, C24 to C32, D6 to D10, D7 to D11, D8 to D12, D9 to D13, J3 to J10, J4 to J9, R10 to R12, R9 to R13, TP7 to TP31
Connections:
- net +3.3V: now also Q5.1 (G), Q6.1 (G), R14.2, R18.2
- net +5V: now also J6.9 (Pin_9), J7.9 (Pin_9), J8.9 (Pin_9), R15.2, R19.2
- net GND: now also J6.10 (Pin_10), J7.10 (Pin_10), J8.10 (Pin_10), R17.1
- net at J10.1 (Pin_1): now also R16.1, R17.2
- net DISP_SDA: now reaches J10.2 (Pin_2)
- net DISP_SDA: now also Q5.2 (S), R14.1
- net DISP_SCL: now reaches J10.3 (Pin_3)
- net DISP_SCL: now also Q6.2 (S), R18.1
- net at U8.1 (PG5): now also TP38.1
- net PB0: now reaches U8.19 (PB0)
- net PB0: now also J7.1 (Pin_1)
- net at U8.2 (PE0): now also TP22.1
- net PB1: now reaches U8.20 (PB1)
- net PB1: now also J7.2 (Pin_2)
- net PB2: now reaches U8.21 (PB2)
- net PB2: now also J7.3 (Pin_3)
- net PB3: now reaches U8.22 (PB3)
- net PB3: now also J7.4 (Pin_4)
- net PB4: now reaches U8.23 (PB4)
- net PB4: now also J7.5 (Pin_5)
- net PB5: now reaches U8.24 (PB5)
- net PB5: now also J7.6 (Pin_6)
- net PB6: now reaches U8.25 (PB6)
- net PB6: now also J7.7 (Pin_7)
- net PB7: now reaches U8.26 (PB7)
- net PB7: now also J7.8 (Pin_8)
- net at U8.28 (PG3): now also TP35.1
- net at U8.29 (PG4): now also TP37.1
- net at U8.3 (PE1): now also TP23.1
- net at U8.4 (PE2): now also TP24.1
- net ATMEGA_SCL: now reaches U8.43 (PD0)
- net ATMEGA_SCL: now also J8.1 (Pin_1), Q6.3 (D), R19.1
- net ATMEGA_SDA: now reaches U8.44 (PD1)
- net ATMEGA_SDA: now also J8.2 (Pin_2), Q5.3 (D), R15.1
- net ATMEGA_Rx: now reaches U8.45 (PD2)
- net ATMEGA_Rx: now also J8.3 (Pin_3)
- net ATMEGA_Tx: now reaches U8.46 (PD3)
- net ATMEGA_Tx: now also J8.4 (Pin_4)
- net AT_DISP_RST: now reaches U8.47 (PD4)
- net AT_DISP_RST: now also J8.5 (Pin_5), R16.2
- net PD5: now reaches U8.48 (PD5)
- net PD5: now also D10.3 (DIN), J8.6 (Pin_6)
- net PD6: now reaches U8.49 (PD6)
- net PD6: now also J8.7 (Pin_7)
- net at U8.5 (PE3): now also TP25.1
- net PD7: now reaches U8.50 (PD7)
- net PD7: now also J8.8 (Pin_8)
- net at U8.53 (PC0): now also TP14.1
- net at U8.54 (PC1): now also TP15.1
- net at U8.55 (PC2): now also TP16.1
- net at U8.56 (PC3): now also TP17.1
- net at U8.57 (PC4): now also TP18.1
- net at U8.58 (PC5): now also TP19.1
- net at U8.59 (PC6): now also TP20.1
- net at U8.6 (PE4): now also TP26.1
- net at U8.60 (PC7): now also TP21.1
- net at U8.7 (PE5): now also TP27.1
- net at U8.70 (PG2): now also TP33.1
- net PA7: now reaches U8.71 (PA7)
- net PA7: now also J6.8 (Pin_8)
- net PA6: now reaches U8.72 (PA6)
- net PA6: now also J6.7 (Pin_7)
- net PA5: now reaches U8.73 (PA5)
- net PA5: now also J6.6 (Pin_6)
- net PA4: now reaches U8.74 (PA4)
- net PA3: now reaches U8.75 (PA3)
- net PA3: now also J6.4 (Pin_4), J6.5 (Pin_5)
- net PA2: now reaches U8.76 (PA2)
- net PA2: now also J6.3 (Pin_3)
- net PA1: now reaches U8.77 (PA1)
- net PA1: now also J6.2 (Pin_2)
- net PA0: now reaches U8.78 (PA0)
- net PA0: now also J6.1 (Pin_1)
- net at U8.8 (PE6): now also TP28.1
- net at U8.9 (PE7): now also TP29.1
- net at U8.94 (PF3): now also TP36.1
- net at U8.95 (PF2): now also TP34.1
- net at U8.96 (PF1): now also TP32.1
- net at U8.97 (PF0): now also TP30.1
- no-connect marks 0 -> 32
Other:
- note added: "Place jumper near power source"
- moved on the sheet: D10, D11, D12, D13, J10, TP31

Commit message: PCB finished
Parts:
- renumbered J8 to J10, J9 to J11, J10 to J12, J6 to J8, J7 to J9, U8 to U9
Connections:
- net PA3: no longer J8.5 (Pin_5)
- net PA4: now also J8.5 (Pin_5)
- net VDDA: now also C27.1, U9.98 (AREF)

Commit message: Prototype PCB finished
Parts:
- Y1: footprint Crystal:Crystal_SMD_ECS_CSM3X-2Pin_7.6x4.1mm -> Crystal:Crystal_SMD_HC49-SD
Connections:
- net VDDA: no longer C27.1, U9.98 (AREF)
- new net: C27.1, U9.98 (AREF)
Other:
- note removed: "Place jumper near power source"
- moved on the sheet: C27
Changed lines of the file:
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@@
 	)
 	(junction
-		(at 73.66 48.26)
-		(diameter 0)
-		(color 0 0 0 0)
-	)
-	(junction
 		(at 78.74 167.64)
 		(diameter 0)
@@
 	(wire
 		(pts
-			(xy 73.66 50.8) (xy 73.66 48.26)
-		)
-		(stroke
-			(width 0)
-			(type default)
-		)
-	)
-	(wire
-		(pts
 			(xy 238.76 43.18) (xy 243.84 43.18)
 		)
@@
 	(wire
 		(pts
-			(xy 73.66 46.99) (xy 73.66 48.26)
-		)
-		(stroke
-			(width 0)
-			(type default)
-		)
-	)
-	(wire
-		(pts
 			(xy 78.74 180.34) (xy 78.74 181.61)
 		)
@@
 		)
 	)
+	(wire
+		(pts
+			(xy 96.52 48.26) (xy 114.3 48.26)
+		)
+		(stroke
+			(width 0)
+			(type default)
+		)
+	)
 	(bus
 		(pts
@@
 	(wire
 		(pts
+			(xy 96.52 49.53) (xy 96.52 48.26)
+		)
+		(stroke
+			(width 0)
+			(type default)
+		)
+	)
+	(wire
+		(pts
 			(xy 398.78 276.86) (xy 398.78 278.13)
 		)
@@
 	(wire
 		(pts
-			(xy 73.66 58.42) (xy 73.66 60.96)
+			(xy 96.52 57.15) (xy 96.52 59.69)
 		)
 		(stroke
@@
 	(wire
 		(pts
-			(xy 73.66 48.26) (xy 114.3 48.26)
-		)
-		(stroke
-			(width 0)
-			(type default)
-		)
-	)
-	(wire
-		(pts
 			(xy 238.76 38.1) (xy 243.84 38.1)
 		)
@@
 		)
 	)
-	(text "Place jumper near power source"
-		(exclude_from_sim no)
-		(at 52.07 60.452 0)
-		(effects
-			(font
-				(size 1.27 1.27)
-			)
-		)
-	)
 	(label "PA0"
 		(at 223.52 38.1 180)
@@
 	(symbol
 		(lib_id "power:GNDREF")
-		(at 73.66 60.96 0)
+		(at 96.52 59.69 0)
 		(unit 1)
 		(exclude_from_sim no)
@@
 		(fields_autoplaced yes)
 		(property "Reference" "#PWR0107"
-			(at 73.66 67.31 0)
+			(at 96.52 66.04 0)
 			(effects
 				(font
@@
 		)
 		(property "Value" "GNDREF"
-			(at 73.66 66.04 0)
+			(at 96.52 64.77 0)
 			(effects
 				(font
@@
 		)
 		(property "Footprint" ""
-			(at 73.66 60.96 0)
+			(at 96.52 59.69 0)
 			(effects
 				(font
@@
 		)
 		(property "Datasheet" ""
-			(at 73.66 60.96 0)
+			(at 96.52 59.69 0)
 			(effects
 				(font
@@
 		)
 		(property "Description" "Power symbol creates a global label with name \"GNDREF\" , reference supply ground"
-			(at 73.66 60.96 0)
+			(at 96.52 59.69 0)
 			(effects
 				(font
@@
 	(symbol
 		(lib_id "Device:C")
-		(at 73.66 54.61 0)
+		(at 96.52 53.34 0)
 		(unit 1)
 		(exclude_from_sim no)
@@
 		(fields_autoplaced yes)
 		(property "Reference" "C27"
-			(at 77.47 53.3399 0)
+			(at 100.33 52.0699 0)
 			(effects
 				(font
@@
 		)
 		(property "Value" "100n"
-			(at 77.47 55.8799 0)
+			(at 100.33 54.6099 0)
 			(effects
 				(font
@@
 		)
 		(property "Footprint" "Capacitor_SMD:C_0805_2012Metric"
-			(at 74.6252 58.42 0)
+			(at 97.4852 57.15 0)
 			(effects
 				(font
@@
 		)
 		(property "Datasheet" "~"
-			(at 73.66 54.61 0)
+			(at 96.52 53.34 0)
 			(effects
 				(font
@@
 		)
 		(property "Description" "Unpolarized capacitor"
-			(at 73.66 54.61 0)
+			(at 96.52 53.34 0)
 			(effects
 				(font
@@
 	)
 	(symbol
-		(lib_id "power:VDDA")
-		(at 73.66 46.99 0)
-		(unit 1)
-		(exclude_from_sim no)
-		(in_bom yes)
-		(on_board yes)
-		(dnp no)
-		(fields_autoplaced yes)
-		(property "Reference" "#PWR0145"
-			(at 73.66 50.8 0)
-			(effects
-				(font
-					(size 1.27 1.27)
-				)
-				(hide yes)
-			)
-		)
-		(property "Value" "VDDA"
-			(at 73.66 41.91 0)
-			(effects
-				(font
-					(size 1.27 1.27)
-				)
-			)
-		)
-		(property "Footprint" ""
-			(at 73.66 46.99 0)
-			(effects
-				(font
-					(size 1.27 1.27)
-				)
-				(hide yes)
-			)
-		)
-		(property "Datasheet" ""
-			(at 73.66 46.99 0)
-			(effects
-				(font
-					(size 1.27 1.27)
-				)
-				(hide yes)
-			)
-		)
-		(property "Description" "Power symbol creates a global label with name \"VDDA\""
-			(at 73.66 46.99 0)
-			(effects
-				(font
-					(size 1.27 1.27)
-				)
-				(hide yes)
-			)
-		)
-		(pin "1"
-		)
-		(instances
-			(project "Automatischer-Kabelschneider"
-				(path "/ff414881-00bc-48a3-bd83-dba8c1da722a/b7d74188-216a-42cc-9b81-f0b98f12fae4"
-					(reference "#PWR0145")
-					(unit 1)
-				)
-			)
-		)
-	)
-	(symbol
 		(lib_id "Connector:TestPoint_Small")
 		(at 156.21 81.28 0)
@@
 			)
 		)
-		(property "Footprint" "Crystal:Crystal_SMD_ECS_CSM3X-2Pin_7.6x4.1mm"
+		(property "Footprint" "Crystal:Crystal_SMD_HC49-SD"
 			(at 96.52 40.64 0)
 			(effects
