File: Hardware/Prototyp/Automatischer-Kabelschneider/powersupply_AKS.kicad_sch (KiCad schematic)
At the start: 4 parts, among them J1 USB_C_Receptacle_USB2.0_16P, U1 AP63203WU, U3 CYPD3177-24LQ

Commit message: 20240410
Parts:
- removed J1: USB_C_Receptacle_USB2.0_16P, Connector_USB:USB_C_Receptacle_GCT_USB4105-xx-A_16P_TopMnt_Horizontal, symbol Connector:USB_C_Receptacle_USB2.0_16P
- removed L1: 3u9, Inductor_SMD:L_Wuerth_MAPI-4020, symbol Device:L
- removed U1: AP63203WU, Package_TO_SOT_SMD:TSOT-23-6, symbol Regulator_Switching:AP63203WU
- removed U3: CYPD3177-24LQ, Package_DFN_QFN:QFN-24-1EP_4x4mm_P0.5mm_EP2.75x2.75mm, symbol Interface_USB:CYPD3177-24LQ
- added C2, C3: 470u, Capacitor_SMD:C_Elec_8x10.2, symbol Device:C_Polarized
- added C5, C8: 1u, Capacitor_SMD:C_0805_2012Metric, symbol Device:C
- added C6, C9: 100n, Capacitor_SMD:C_0805_2012Metric, symbol Device:C
- added C7: 3u3, Capacitor_SMD:C_0805_2012Metric, symbol Device:C
- added D1: LED, Diode_SMD:D_0805_2012Metric, symbol Device:LED
- added D2, D3, D4, D5: D_TVS, Diode_SMD:D_0603_1608Metric, symbol Device:D_TVS
- added J1: Conn_01x04, Connector_Phoenix_GMSTB:PhoenixContact_GMSTBA_2,5_4-G-7,62_1x04_P7.62mm_Horizontal, symbol Connector_Generic:Conn_01x04
- added J2: USB_C_Receptacle_USB2.0_16P, Connector_USB:USB_C_Receptacle_GCT_USB4105-xx-A_16P_TopMnt_Horizontal, symbol Connector:USB_C_Receptacle_USB2.0_16P
- added R1, R2: 1k, Resistor_SMD:R_0805_2012Metric, symbol Device:R
- added R5, R6: 5k1, Resistor_SMD:R_0805_2012Metric, symbol Device:R
- added U1: CYPD3177-24LQ, Package_DFN_QFN:QFN-24-1EP_4x4mm_P0.5mm_EP2.75x2.75mm, symbol Interface_USB:CYPD3177-24LQ
- added U5: TVS220x, Package_SON:WSON-6-1EP_2x2mm_P0.65mm_EP1x1.6mm, symbol Power_Protection:TVS2200DRV
Connections:
- new net: R2.1, U1.10 (FLIP)
- new net: R5.2, R6.1, U1.5 (ISNK_COARSE)
- new net: D1.1 (K), U1.9 (FAULT)
- new net: D1.2 (A), R1.1
- new net +20V: C2.1, J1.1 (Pin_1)
- new net +3.3V: C3.1, J1.3 (Pin_3)
- new net CC1: D2.2 (A2), J2.A5 (CC1), U1.15 (CC1)
- new net CC2: D3.2 (A2), J2.B5 (CC2), U1.14 (CC2)
- new net D+: D5.2 (A2), J2.A6 (D+), J2.B6 (D+)
- new net D-: D4.2 (A2), J2.A7 (D-), J2.B7 (D-)
- new net GND: C2.2, C3.2, C5.2, C6.2, C7.2, C8.2, C9.2, D2.1 (A1), D3.1 (A1), D4.1 (A1), D5.1 (A1), J1.2 (Pin_2), J1.4 (Pin_4), J2.A1 (GND), J2.A12 (GND), J2.B1 (GND), J2.B12 (GND), R6.2, U1.19 (GND), U1.22 (GND), U1.25 (GND), U1.6 (ISNK_FINE), U5.1 (GND), U5.2 (GND), U5.3 (GND), U5.7 (GND)
- new net VBUS: C7.1, J2.A4 (VBUS), J2.A9 (VBUS), J2.B4 (VBUS), J2.B9 (VBUS), U1.18 (VBUS_IN), U5.4 (IN), U5.5 (IN), U5.6 (IN)
- new net VCCD: C5.1, U1.24 (VCCD)
- new net VDDD: C6.1, C8.1, C9.1, R1.2, R2.2, R5.1, U1.1 (VBUS_MIN), U1.2 (VBUS_MAX), U1.23 (VDDD)
- no-connect marks 0 -> 7

Commit message: 20240411
Parts:
- removed C3: 470u, Capacitor_SMD:C_Elec_8x10.2, symbol Device:C_Polarized
- removed R2: 1k, Resistor_SMD:R_0805_2012Metric, symbol Device:R
- added C10, C11: 1u, Capacitor_SMD:C_0805_2012Metric, symbol Device:C
- added C12, C13: 22u, Capacitor_SMD:C_0805_2012Metric, symbol Device:C
- added C14: 100n, Capacitor_SMD:C_0805_2012Metric, symbol Device:C
- added C3: 10u, Capacitor_SMD:C_0805_2012Metric, symbol Device:C
- added L1: 3u9, Inductor_SMD_Wurth:L_Wurth_WE-LQSH-4020, symbol Device:L
- added Q1, Q2: IRF540N, Package_TO_SOT_THT:TO-220-3_Horizontal_TabDown, symbol Transistor_FET:IRF540N
- added R3: 10k, Resistor_SMD:R_0805_2012Metric, symbol Device:R
- added R4: 50k, Resistor_SMD:R_0805_2012Metric, symbol Device:R
- added R7: 1k, Resistor_SMD:R_0805_2012Metric, symbol Device:R
- added U3: AP63203WU, Package_TO_SOT_SMD:TSOT-23-6, symbol Regulator_Switching:AP63203WU
- D1: value LED -> gr
Connections:
- net +20V: now also J1.2 (Pin_2), U1.11 (VDC_OUT), C11.1, C3.1, Q2.2 (D), U3.2 (EN), U3.3 (IN); no longer J1.1 (Pin_1)
- net +3.3V: now also C12.1, C13.1, L1.2, U3.1 (FB)
- net GND: now also C12.2, C13.2, C3.2, U3.4 (GND); no longer J1.2 (Pin_2)
- net VBUS: now also J1.1 (Pin_1), C10.1, Q1.2 (D), R3.1
- net at U1.3 (VBUS_FET_EN): now also R7.2
- new net: C14.1, L1.1, U3.5 (SW)
- new net: C14.2, U3.6 (BST)
- new net: Q1.3 (S), Q2.3 (S), R4.1
- new net GATE: C10.2, C11.2, Q1.1 (G), Q2.1 (G), R3.2, R4.2, R7.1
- no-connect marks 7 -> 9
Other:
- moved on the sheet: C2, C5, C6, C7, C8, C9, D1, D2, D3, D4, D5, J1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

Commit message: 20240415
Parts:
- added H1, H2, H3, H4: MountingHole, MountingHole:MountingHole_3.2mm_M3, symbol Mechanical:MountingHole
- added TP1, TP2, TP3, TP4, TP5, TP6: TestPoint_Small, TestPoint:TestPoint_Pad_D1.0mm, symbol Connector:TestPoint_Small
- renumbered C10 to C1, C3 to C10, C12 to C11, C13 to C12, C11 to C2, C5 to C3, C7 to C4, C8 to C5, C9 to C7, C2 to C8, C14 to C9, J2 to J1, J1 to J2, R5 to R1, R3 to R2, R4 to R3, R6 to R4, R7 to R5, R1 to R6, U5 to U1, U1 to U2
Connections:
- net at U2.10 (FLIP): now also TP1.1
- net at U2.12 (HPI_SDA): now also TP3.1
- net at U2.13 (HPI_SCL): now also TP2.1
- net at U2.4 (SAFE_PWR_EN): now also TP5.1
- net at U2.7 (~{HPI_INT}): now also TP4.1
- net at U2.8 (GPIO_1): now also TP6.1
- no-connect marks 9 -> 3
Other:
- moved on the sheet: U1

Commit message: 20240418
Parts:
- added C16: 100n, Capacitor_SMD:C_0805_2012Metric, symbol Device:C
- added C17: 10u, Capacitor_SMD:C_0805_2012Metric, symbol Device:C
- added C18, C19: 22u, Capacitor_SMD:C_0805_2012Metric, symbol Device:C
- added L2: 4u7, Inductor_SMD_Wurth:L_Wurth_WE-LQSH-4020, symbol Device:L
- added U7: AP63205WU, Package_TO_SOT_SMD:TSOT-23-6, symbol Regulator_Switching:AP63205WU
Connections:
- net +20V: now also J2.1 (Pin_1), C17.1, U7.2 (EN), U7.3 (IN); no longer J2.2 (Pin_2)
- net GND: now also C17.2, C18.2, C19.2, U7.4 (GND)
- net VBUS: no longer J2.1 (Pin_1)
- net VBUS_FET_EN: now reaches R5.2, U2.3 (VBUS_FET_EN)
- net ISNK_COARSE: now reaches R1.2, R4.1, U2.5 (ISNK_COARSE)
- new net: C16.1, L2.1, U7.5 (SW)
- new net: C16.2, U7.6 (BST)
- new net +5V: C18.1, C19.1, J2.2 (Pin_2), L2.2, U7.1 (FB)
Other:
- moved on the sheet: C1, C10, C11, C12, C2, C3, C4, C5, C6, C7, C8, C9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

Commit message: 20240501
Changed lines of the file:
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@@
 		(on_board yes)
 		(dnp no)
-		(fields_autoplaced yes)
 		(property "Reference" "#PWR033"
 			(at 146.05 140.97 0)
@@
 		)
 		(property "Value" "+5V"
-			(at 146.05 132.08 0)
+			(at 146.05 132.08 90)
 			(effects
 				(font
@@
 		(on_board yes)
 		(dnp no)
-		(fields_autoplaced yes)
 		(property "Reference" "#PWR035"
 			(at 149.86 140.97 0)
@@
 		)
 		(property "Value" "+3.3V"
-			(at 152.4 135.8899 0)
+			(at 149.86 131.064 90)
 			(effects
 				(font
 					(size 1.27 1.27)
 				)
-				(justify left)
 			)
 		)
@@
 		(on_board yes)
 		(dnp no)
-		(fields_autoplaced yes)
 		(property "Reference" "#PWR034"
 			(at 142.24 140.97 0)
@@
 		)
 		(property "Value" "+20V"
-			(at 142.24 132.08 0)
+			(at 142.24 132.08 90)
 			(effects
 				(font

Commit message: Schematic completed
Parts:
- removed C8: 470u, Capacitor_SMD:C_Elec_8x10.2, symbol Device:C_Polarized
- renumbered C11 to C10, C12 to C11, C16 to C12, C17 to C13, C18 to C14, C19 to C15, C9 to C8, C10 to C9, U7 to U4

Commit message: PCB finished
Parts:
- added U1: TVS220x, Package_SON:WSON-6-1EP_2x2mm_P0.65mm_EP1x1.6mm, symbol Power_Protection:TVS2200DRV
- Q1, Q2: footprint Package_TO_SOT_THT:TO-220-3_Horizontal_TabDown -> Package_TO_SOT_THT:TO-220-3_Vertical
- renumbered U1 to U2, U2 to U3, U3 to U4, U4 to U5
Connections:
- net GND: now also U1.1 (GND), U1.2 (GND), U1.3 (GND), U1.7 (GND)
- net VBUS: now also U1.4 (IN), U1.5 (IN), U1.6 (IN)
Other:
- moved on the sheet: U2

Commit message: Changed Q1 & Q2 from NMOS to PMOS
Parts:
- Q1, Q2: symbol Transistor_FET:IRF540N -> Simulation_SPICE:PMOS
Connections:
- net +20V: now also Q2.1 (D); no longer Q2.2 (D)
- net GATE: now also Q1.2 (G), Q2.2 (G); no longer Q1.1 (G), Q2.1 (G)
- net VBUS: now also Q1.1 (D); no longer Q1.2 (D)
Other:
- note added: "P kanal!!!!!"
Changed lines of the file:
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@@
 		)
 	)
+	(text "P kanal!!!!!"
+		(exclude_from_sim no)
+		(at 216.154 22.098 0)
+		(effects
+			(font
+				(size 1.27 1.27)
+			)
+		)
+	)
 	(label "GATE"
 		(at 228.6 44.45 0)
@@
 	)
 	(symbol
-		(lib_id "Transistor_FET:IRF540N")
+		(lib_id "Simulation_SPICE:PMOS")
 		(at 218.44 35.56 90)
 		(unit 1)
@@
 		)
 		(property "Footprint" "Package_TO_SOT_THT:TO-220-3_Vertical"
-			(at 220.345 30.48 0)
+			(at 215.9 30.48 0)
 			(effects
 				(font
 					(size 1.27 1.27)
-					(italic yes)
 				)
-				(justify left)
 				(hide yes)
 			)
 		)
-		(property "Datasheet" "http://www.irf.com/product-info/datasheets/data/irf540n.pdf"
-			(at 222.25 30.48 0)
+		(property "Datasheet" "https://ngspice.sourceforge.io/docs/ngspice-html-manual/manual.xhtml#cha_MOSFETs"
+			(at 231.14 35.56 0)
 			(effects
 				(font
 					(size 1.27 1.27)
 				)
-				(justify left)
 				(hide yes)
 			)
 		)
-		(property "Description" "33A Id, 100V Vds, HEXFET N-Channel MOSFET, TO-220"
+		(property "Description" "P-MOSFET transistor, drain/source/gate"
 			(at 218.44 35.56 0)
 			(effects
@@
 			)
 		)
+		(property "Sim.Device" "PMOS"
+			(at 235.585 35.56 0)
+			(effects
+				(font
+					(size 1.27 1.27)
+				)
+				(hide yes)
+			)
+		)
+		(property "Sim.Type" "VDMOS"
+			(at 237.49 35.56 0)
+			(effects
+				(font
+					(size 1.27 1.27)
+				)
+				(hide yes)
+			)
+		)
+		(property "Sim.Pins" "1=D 2=G 3=S"
+			(at 233.68 35.56 0)
+			(effects
+				(font
+					(size 1.27 1.27)
+				)
+				(hide yes)
+			)
+		)
 		(pin "1"
 		)
@@
 	)
 	(symbol
-		(lib_id "Transistor_FET:IRF540N")
+		(lib_id "Simulation_SPICE:PMOS")
 		(at 240.03 35.56 270)
 		(mirror x)
@@
 		)
 		(property "Footprint" "Package_TO_SOT_THT:TO-220-3_Vertical"
-			(at 238.125 30.48 0)
+			(at 242.57 30.48 0)
 			(effects
 				(font
 					(size 1.27 1.27)
-					(italic yes)
 				)
-				(justify left)
 				(hide yes)
 			)
 		)
-		(property "Datasheet" "http://www.irf.com/product-info/datasheets/data/irf540n.pdf"
-			(at 236.22 30.48 0)
+		(property "Datasheet" "https://ngspice.sourceforge.io/docs/ngspice-html-manual/manual.xhtml#cha_MOSFETs"
+			(at 227.33 35.56 0)
 			(effects
 				(font
 					(size 1.27 1.27)
 				)
-				(justify left)
 				(hide yes)
 			)
 		)
-		(property "Description" "33A Id, 100V Vds, HEXFET N-Channel MOSFET, TO-220"
+		(property "Description" "P-MOSFET transistor, drain/source/gate"
 			(at 240.03 35.56 0)
 			(effects
 				(font
+					(size 1.27 1.27)
+				)
+				(hide yes)
+			)
+		)
+		(property "Sim.Device" "PMOS"
+			(at 222.885 35.56 0)
+			(effects
+				(font
+					(size 1.27 1.27)
+				)
+				(hide yes)
+			)
+		)
+		(property "Sim.Type" "VDMOS"
+			(at 220.98 35.56 0)
+			(effects
+				(font
+					(size 1.27 1.27)
+				)
+				(hide yes)
+			)
+		)
+		(property "Sim.Pins" "1=D 2=G 3=S"
+			(at 224.79 35.56 0)
+			(effects
+				(font
