File: Hardware/v1.0/Mainboard/Main.kicad_sch (KiCad schematic)
At the start: 20 parts, among them J1 Conn_01x04, J2 Conn_02x02_Odd_Even, J3 Conn_01x04, J4 Conn_02x03_Odd_Even, J5 Conn_02x03_Odd_Even, J6 Conn_02x03_Odd_Even, SW1 SW_Push, SW2 SW_Push, U3 TMC2209_SILENTSTEPSTICK, U4 ESP32-S3-WROOM-2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

Commit message: finished pcb v1.0
Changed lines of the file:
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@@
 	(bus
 		(pts
-			(xy 128.27 77.47) (xy 128.27 78.74)
+			(xy 128.27 78.74) (xy 128.27 77.47)
 		)
 		(stroke
