File: Hardware/v1.0/Mainboard/PSU.kicad_sch (KiCad schematic)
At the start: 9 parts, among them U1 AP63203WU

Commit message: finished pcb v1.0
Changed lines of the file:
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@@
+	)
+	(junction
+		(at 119.38 80.01)
+		(diameter 0)
+		(color 0 0 0 0)
 	)
 	(junction
@@
 	)
 	(junction
-		(at 120.65 80.01)
-		(diameter 0)
-		(color 0 0 0 0)
-	)
-	(junction
 		(at 116.84 85.09)
 		(diameter 0)
@@
 	(wire
 		(pts
-			(xy 115.57 90.17) (xy 120.65 90.17)
+			(xy 115.57 90.17) (xy 119.38 90.17)
 		)
 		(stroke
@@
 	(wire
 		(pts
-			(xy 120.65 80.01) (xy 125.73 80.01)
-		)
-		(stroke
-			(width 0)
-			(type default)
-		)
-	)
-	(wire
-		(pts
 			(xy 227.33 91.44) (xy 228.6 91.44)
 		)
@@
 	(wire
 		(pts
-			(xy 115.57 87.63) (xy 123.19 87.63)
+			(xy 115.57 87.63) (xy 121.92 87.63)
 		)
 		(stroke
@@
 	(wire
 		(pts
+			(xy 119.38 80.01) (xy 125.73 80.01)
+		)
+		(stroke
+			(width 0)
+			(type default)
+		)
+	)
+	(wire
+		(pts
 			(xy 201.93 88.9) (xy 207.01 88.9)
 		)
@@
 	(wire
 		(pts
-			(xy 123.19 87.63) (xy 123.19 90.17)
+			(xy 121.92 87.63) (xy 121.92 90.17)
 		)
 		(stroke
@@
 	(wire
 		(pts
-			(xy 120.65 90.17) (xy 120.65 80.01)
+			(xy 119.38 90.17) (xy 119.38 80.01)
 		)
 		(stroke
@@
 	(wire
 		(pts
-			(xy 115.57 80.01) (xy 120.65 80.01)
-		)
-		(stroke
-			(width 0)
-			(type default)
-		)
-	)
-	(wire
-		(pts
-			(xy 123.19 90.17) (xy 125.73 90.17)
-		)
-		(stroke
+			(xy 115.57 80.01) (xy 119.38 80.01)
+		)
+		(stroke
+			(width 0)
+			(type default)
+		)
+	)
+	(wire
+		(pts
+			(xy 121.92 90.17) (xy 125.73 90.17)
+		)
+		(stroke
