File: Hardware/v1.0/Mainboard/Mainboard.kicad_pcb (KiCad board)
At the start: 2 copper layers, 33 parts, among them J1 Conn_01x04, J2 Conn_02x02_Odd_Even, J3 Conn_01x04, J4 Conn_02x03_Odd_Even, J5 Conn_02x03_Odd_Even, J6 Conn_02x03_Odd_Even, SW1 SW_Push, SW2 SW_Push, U1 AP63203WU, U3 TMC2209_SILENTSTEPSTICK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

Commit message: finished pcb v1.0
Parts:
- moved J6 148.6 mm to (186.4, 112.3)
- moved J5 142.9 mm to (186.4, 122.3)
- moved J2 138.0 mm to (186.4, 104.9)
- moved JP1 124.8 mm to (181.6, 121.9), turned to 180 degrees
- moved J4 119.1 mm to (172.1, 94.5), turned to -90 degrees
- moved H2 111.2 mm to (97.6, 133.6)
- moved J3 93.3 mm to (132.6, 130.4)
- moved H1 80.6 mm to (97.6, 68.6)
- moved J1 76.3 mm to (112.6, 130.4)
- moved H3 73.1 mm to (187.6, 133.6)
- moved C11 64.7 mm to (149.3, 124.2), turned to 180 degrees
- moved U2 63.2 mm to (117.6, 81.3), turned to -90 degrees
- moved C10 57.6 mm to (133.5, 124.7), turned to 180 degrees
- moved U5 56.9 mm to (141.1, 114.9), turned to 90 degrees
- moved C8 48.9 mm to (111.2, 124.7), turned to 180 degrees
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Routing:
- net +3.3V: track 0.00 -> 274.3 mm, vias 0 -> 6
- net +20V: track 0.00 -> 158.8 mm
- net SERVO2: track 0.00 -> 77.8 mm, vias 0 -> 1
- net /Main Sheet/MD1_DIR: track 0.00 -> 67.6 mm, vias 0 -> 1
- net /Main Sheet/MD1_STEP: track 0.00 -> 63.8 mm, vias 0 -> 1
- net SERVO1: track 0.00 -> 63.3 mm, vias 0 -> 1
- net WS2812: track 0.00 -> 56.4 mm, vias 0 -> 2
- net /Main Sheet/MD1_!EN: track 0.00 -> 52.2 mm, vias 0 -> 1
- net /Main Sheet/EN: track 0.00 -> 50.4 mm, vias 0 -> 2
- net /Main Sheet/MD1_MS1: track 0.00 -> 50.1 mm, vias 0 -> 1
- net /Main Sheet/MD1_MS2: track 0.00 -> 49.3 mm, vias 0 -> 1
- net IO2: track 0.00 -> 47.9 mm, vias 0 -> 1
- net IO1: track 0.00 -> 45.7 mm, vias 0 -> 1
- net /Main Sheet/MD2_DIR: track 0.00 -> 44.4 mm, vias 0 -> 2
- net GND: track 0.00 -> 43.7 mm, vias 0 -> 83
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- added copper zone on F.Cu, net +20V
- added copper zone on F.Cu, net +3.3V
- added copper zone on B.Cu, net GND
- added copper zone on F.Cu, net GND
- added copper zone on F.Cu, net Net-(U1-SW)
Other:
- board outline added: 100 x 75 mm
- board text added: "+3V3 GND"
- board text added: "+3V3 WS2812 GND"
- board text added: "+3V3|+20V"
- board text added: "AKS v1.0"
- board text added: "BOOT"
- board text added: "ENABLE"
- board text added: "ID2 ID1 ID0"
- board text added: "IO1 IO2 GND"
- board text added: "MD1_M1A MD1_M1B MD1_M2A MD1_M2B"
- board text added: "MD2_M1A MD2_M1B MD2_M2A MD2_M2B"
- board text added: "Tx Rx"
- board text added: "V+ SERVO1 GND"
- board text added: "V+ SERVO2 GND"

Commit message: Gerber created
Routing:
- net GND: vias 83 -> 86
Changed lines of the file:
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@@
 		(tags "capacitor")
 		(property "Reference" "C2"
-			(at -2.794 0 360)
+			(at -2.794 0 0)
 			(layer "F.SilkS")
 			(effects
@@
 		)
 		(property "Value" "10u"
-			(at 0 1.68 360)
+			(at 0 1.68 0)
 			(layer "F.Fab")
 			(effects
@@
 		)
 		(fp_text user "${REFERENCE}"
-			(at 0 0 360)
+			(at 0 0 0)
 			(layer "F.Fab")
 			(effects
@@
 		(tags "capacitor")
 		(property "Reference" "C3"
-			(at 2.794 0 360)
+			(at 2.794 0 0)
 			(layer "F.SilkS")
 			(effects
@@
 		)
 		(property "Value" "22u"
-			(at 0 1.68 360)
+			(at 0 1.68 0)
 			(layer "F.Fab")
 			(effects
@@
 		)
 		(fp_text user "${REFERENCE}"
-			(at 0 0 360)
+			(at 0 0 0)
 			(layer "F.Fab")
 			(effects
@@
 		(at 118.646 114.87 90)
 		(property "Reference" "U3"
-			(at -5.075 -11.155 270)
+			(at -5.075 -11.155 -90)
 			(layer "F.SilkS")
 			(hide yes)
@@
 		)
 		(property "Value" "TMC2209_SILENTSTEPSTICK"
-			(at 11.05 11.115 270)
+			(at 11.05 11.115 -90)
 			(layer "F.Fab")
 			(effects
@@
 		(at 141.146 114.87 90)
 		(property "Reference" "U5"
-			(at -5.075 -11.155 270)
+			(at -5.075 -11.155 -90)
 			(layer "F.SilkS")
 			(hide yes)
@@
 		)
 		(property "Value" "TMC2209_SILENTSTEPSTICK"
-			(at 11.05 11.115 270)
+			(at 11.05 11.115 -90)
 			(layer "F.Fab")
 			(effects
@@
 		(tags "TSOT TO_SOT_SMD")
 		(property "Reference" "U1"
-			(at -3.048 0 360)
+			(at -3.048 0 0)
 			(layer "F.SilkS")
 			(effects
@@
 		)
 		(property "Value" "AP63203WU"
-			(at 0 2.4 360)
+			(at 0 2.4 0)
 			(layer "F.Fab")
 			(effects
@@
 		)
 		(fp_text user "${REFERENCE}"
-			(at 0 0 360)
+			(at 0 0 0)
 			(layer "F.Fab")
 			(effects
@@
 		(tags "capacitor")
 		(property "Reference" "C4"
-			(at 2.794 0 360)
+			(at 2.794 0 0)
 			(layer "F.SilkS")
 			(effects
@@
 		)
 		(property "Value" "22u"
-			(at 0 1.68 360)
+			(at 0 1.68 0)
 			(layer "F.Fab")
 			(effects
@@
 		)
 		(fp_text user "${REFERENCE}"
-			(at 0 0 360)
+			(at 0 0 0)
 			(layer "F.Fab")
 			(effects
@@
 	)
 	(via
+		(at 146.304 86.868)
+		(size 0.6)
+		(drill 0.3)
+		(layers "F.Cu" "B.Cu")
+		(net 3)
+	)
+	(via
 		(at 133 137)
 		(size 0.6)
@@
 	)
 	(via
+		(at 137.16 83.312)
+		(size 0.6)
+		(drill 0.3)
+		(layers "F.Cu" "B.Cu")
+		(net 3)
+	)
+	(via
 		(at 178.816 92.964)
 		(size 0.6)
@@
 		(size 0.6)
 		(drill 0.3)
+		(layers "F.Cu" "B.Cu")
+		(net 3)
+	)
+	(via
+		(at 173.228 112.268)
+		(size 0.6)
+		(drill 0.3)
